File: src/Morfeas_RPi_Hat/Hardware/Morfeas_Rpi_Hat.sch (KiCad schematic (older format))
At the start: 0 parts

Commit message: Update
Parts:
- added J?: RPi_header, symbol Connector_Generic:Conn_02x20_Odd_Even
Changed lines of the file:
@@
 Comment4 "Author: Sam Harry Tzavaras"
 $EndDescr
+$Comp
+L Connector_Generic:Conn_02x20_Odd_Even J?
+U 1 1 5E041881
+P 2150 4000
+F 0 "J?" H 2200 5117 50  0000 C CNN
+F 1 "RPi_header" H 2200 5026 50  0000 C CNN
+F 2 "" H 2150 4000 50  0001 C CNN
+F 3 "~" H 2150 4000 50  0001 C CNN
+	1    2150 4000
+	1    0    0    -1
+$EndComp
+$Comp
+L power:+5V #PWR?
+U 1 1 5E047DD2
+P 2600 3000
+F 0 "#PWR?" H 2600 2850 50  0001 C CNN
+F 1 "+5V" H 2615 3173 50  0000 C CNN
+F 2 "" H 2600 3000 50  0001 C CNN
+F 3 "" H 2600 3000 50  0001 C CNN
+	1    2600 3000
+	1    0    0    -1
+$EndComp
+$Comp
+L power:GND #PWR?
+U 1 1 5E048E34
+P 2950 3800
+F 0 "#PWR?" H 2950 3550 50  0001 C CNN
+F 1 "GND" H 2955 3627 50  0000 C CNN
+F 2 "" H 2950 3800 50  0001 C CNN
+F 3 "" H 2950 3800 50  0001 C CNN
+	1    2950 3800
+	1    0    0    -1
+$EndComp
 $EndSCHEMATC

Commit message: Update
Parts:
- added BT?: Battery_Cell, symbol Device:Battery_Cell
- added C?: 100nf, symbol Device:C_Small
- added D?: D_ALT, symbol Device:D_ALT
- added J?: Conn_01x03_Female, symbol Connector:Conn_01x03_Female
- added Q?: Q_PMOS_GDS, symbol Device:Q_PMOS_GDS
- added R?: 22mΩ, symbol Device:R_US
- added U?: DS3231SN#T&R, SOIC127P1032X265-16N, symbol Morfeas_Rpi_Hat:DS3231SN#T&R
- added U?: TLV70433DBVT, DBV5, symbol Morfeas_Rpi_Hat:TLV70433DBVT
- added U?: SP3232EET-L, SOIC127P1030X265-16N, symbol Morfeas_Rpi_Hat:SP3232EET-L
- added U?: 24AA08T-I_OT, SOT-23-5_MC, symbol Morfeas_Rpi_Hat:24AA08T-I_OT
- added U?: MAX9611AUB+, 21-0061L, symbol Morfeas_Rpi_Hat:MAX9611AUB+
Connections:
- net labels added: +24V, +3.3V, SCL, SDA
- wire segments 0 -> 33

Commit message: Update
Parts:
- added C1: 10uF, Capacitor_SMD:C_1206_3216Metric, symbol Device:C_Small
- added C10, C11, C12, C14, C4, C5, C7, C8, C9: 100nf, Capacitor_SMD:C_0805_2012Metric, symbol Device:C_Small
- added C2, C3, C6: 10uf, Capacitor_SMD:C_1206_3216Metric, symbol Device:C_Small
- added D2, D3: Zener10V, Diode_THT:D_DO-35_SOD27_P7.62mm_Horizontal, symbol Device:D_Zener_ALT
- added H1, H2, H3, H4: MountingHole, MountingHole:MountingHole_3mm, symbol Mechanical:MountingHole
- added J1: Power IN, symbol Connector:Conn_01x03_Female
- added J4: CAN1_Power+, symbol Connector:Conn_01x03_Female
- added L1: 10uH, Inductor_THT:L_Axial_L6.6mm_D2.7mm_P10.16mm_Horizontal_Vishay_IM-2, symbol Device:L
- added Q2: Q_PMOS_GDS, Package_TO_SOT_SMD:TO-263-2, symbol Device:Q_PMOS_GDS
- added R10, R9: 2.2kΩ, Resistor_SMD:R_1206_3216Metric, symbol Device:R_US
- added R2: 22mΩ, Resistor_SMD:R_2512_6332Metric, symbol Device:R_US
- added R3, R4: 1.3kΩ, Resistor_SMD:R_1206_3216Metric, symbol Device:R_US
- added R5, R6: 18kΩ, Resistor_SMD:R_1206_3216Metric, symbol Device:R_US
- added R7, R8: 1.2kΩ, Resistor_SMD:R_1206_3216Metric, symbol Device:R_US
- added U2: TSR2-2450, Morfeas_RPi_Hat:TSR2-2450, symbol Regulator_Linear:L7805
- added U7: MAX9611, Morfeas_RPi_Hat:MAX9611AUB&plus_, symbol Morfeas_Rpi_Hat:MAX9611AUB+
- BT1: renamed from BT?; footprint (none) -> Battery:BatteryHolder_Keystone_106_1x20mm
- C13: renamed from C?; footprint (none) -> Capacitor_SMD:C_0805_2012Metric
- D1: renamed from D?; value D_ALT -> 1N4007; footprint (none) -> Diode_THT:D_DO-34_SOD68_P7.62mm_Horizontal
- J2: renamed from J?; footprint (none) -> Connector_PinSocket_2.54mm:PinSocket_2x20_P2.54mm_Vertical
- J3: renamed from J?; value Conn_01x03_Female -> CAN0_Power+
- Q1: renamed from Q?; footprint (none) -> Package_TO_SOT_SMD:TO-263-2
- R1: renamed from R?; footprint (none) -> Resistor_SMD:R_2512_6332Metric
- U1: renamed from U?; value DS3231SN#T&R -> DS3231; footprint SOIC127P1032X265-16N -> Project's_libs:SOIC127P1032X265-16N
- U3: renamed from U?; value TLV70433DBVT -> TLV70433; footprint DBV5 -> Morfeas_RPi_Hat:24AA08T-I&slash_OT
- U4: renamed from U?; value SP3232EET-L -> SP3232; footprint SOIC127P1030X265-16N -> Package_SO:SOIC-16_3.9x9.9mm_P1.27mm; symbol Morfeas_Rpi_Hat:SP3232EET-L -> Morfeas_Rpi_Hat:SP3232
- U5: renamed from U?; value 24AA08T-I_OT -> 24AA08; footprint SOT-23-5_MC -> Morfeas_RPi_Hat:24AA08T-I&slash_OT
- U6: renamed from U?; value MAX9611AUB+ -> MAX9611; footprint 21-0061L -> Morfeas_RPi_Hat:MAX9611AUB&plus_
Connections:
- net labels added: RXD, TXD
- wire segments 33 -> 131
- no-connect marks 0 -> 15
Other:
- note added: "Power Supply Unit"
- note added: "Power module (CAN0)"
- note added: "Power module (CAN1)"
- moved on the sheet: C13, D1, J3, Q1, R1, U3, U5, U6

Commit message: Update
Parts:
- BT1: footprint Battery:BatteryHolder_Keystone_106_1x20mm -> Battery:BatteryHolder_Keystone_103_1x20mm
Changed lines of the file:
@@
 F 0 "BT1" H 3568 6696 50  0000 L CNN
 F 1 "Battery_Cell" H 3568 6605 50  0000 L CNN
-F 2 "Battery:BatteryHolder_Keystone_106_1x20mm" V 3450 6660 50  0001 C CNN
+F 2 "Battery:BatteryHolder_Keystone_103_1x20mm" V 3450 6660 50  0001 C CNN
 F 3 "~" V 3450 6660 50  0001 C CNN
 	1    3450 6600

Commit message: Update, add some 3d_models
Parts:
- added J5: RS_232, Connectors_Molex:Molex_KK-6410-03_03x2.54mm_Straight, symbol Connector:Conn_01x03_Male
- J1, J3, J4: footprint (none) -> Morfeas_RPi_hat:SPTH_V1,5
- Q1, Q2: value Q_PMOS_GDS -> SUM110P06
- U2: footprint Morfeas_RPi_Hat:TSR2-2450 -> Morfeas_RPi_hat:TSR2-2450
- U3: footprint Morfeas_RPi_Hat:24AA08T-I&slash_OT -> Morfeas_RPi_hat:TLV70433DBVT
Connections:
- net GND: now also J5.3 (Pin_3)
- net at U4.13 (R1IN): now also J5.2 (Pin_2)
- net at U4.14 (T1OUT): now also J5.1 (Pin_1)
Changed lines of the file:
@@
-$EndComp
-$Comp
-L Morfeas_Rpi_Hat:TLV70433DBVT U3
-U 1 1 5E056599
-P 3600 1050
-F 0 "U3" H 3300 1350 60  0000 L CNN
-F 1 "TLV70433" H 3300 1250 60  0000 L CNN
-F 2 "Morfeas_RPi_Hat:24AA08T-I&slash_OT" H 4100 900 60  0001 C CNN
-F 3 "" H 3000 1300 60  0000 C CNN
-	1    3600 1050
-	1    0    0    -1
 $EndComp
 $Comp
@@
 F 0 "J3" H 7892 1435 50  0000 C CNN
 F 1 "CAN0_Power+" H 7892 1344 50  0000 C CNN
-F 2 "" H 8000 1150 50  0001 C CNN
+F 2 "Morfeas_RPi_hat:SPTH_V1,5" H 8000 1150 50  0001 C CNN
 F 3 "~" H 8000 1150 50  0001 C CNN
 	1    8000 1150
@@
 P 10150 1250
 F 0 "Q1" V 10492 1250 50  0000 C CNN
-F 1 "Q_PMOS_GDS" V 10401 1250 50  0000 C CNN
+F 1 "SUM110P06" V 10401 1250 50  0000 C CNN
 F 2 "Package_TO_SOT_SMD:TO-263-2" H 10350 1350 50  0001 C CNN
 F 3 "~" H 10150 1250 50  0001 C CNN
@@
 P 10150 3900
 F 0 "Q2" V 10492 3900 50  0000 C CNN
-F 1 "Q_PMOS_GDS" V 10401 3900 50  0000 C CNN
+F 1 "SUM110P06" V 10401 3900 50  0000 C CNN
 F 2 "Package_TO_SOT_SMD:TO-263-2" H 10350 4000 50  0001 C CNN
 F 3 "~" H 10150 3900 50  0001 C CNN
@@
 F 0 "J1" H 750 1300 50  0000 C CNN
 F 1 "Power IN" V 900 1100 50  0000 C CNN
-F 2 "" H 800 1100 50  0001 C CNN
+F 2 "Morfeas_RPi_hat:SPTH_V1,5" H 800 1100 50  0001 C CNN
 F 3 "~" H 800 1100 50  0001 C CNN
 	1    800  1100
@@
 F 0 "U2" H 2400 1250 50  0000 C CNN
 F 1 "TSR2-2450" H 2550 1151 50  0000 C CNN
-F 2 "Morfeas_RPi_Hat:TSR2-2450" H 2575 850 50  0001 L CIN
-F 3 "https://assets.tracopower.com/20191223103541/TSR2/documents/tsr2-datasheet.pdf" H 2550 950 50  0001 C CNN
+F 2 "Morfeas_RPi_hat:TSR2-2450" H 2575 850 50  0001 L CIN
+F 3 "http://www.st.com/content/ccc/resource/technical/document/datasheet/41/4f/b3/b0/12/d4/47/88/CD00000444.pdf/files/CD00000444.pdf/jcr:content/translations/en.CD00000444.pdf" H 2550 950 50  0001 C CNN
 	1    2550 1000
 	1    0    0    -1
@@
 F 0 "J4" H 7892 4085 50  0000 C CNN
 F 1 "CAN1_Power+" H 7892 3994 50  0000 C CNN
-F 2 "" H 8000 3800 50  0001 C CNN
+F 2 "Morfeas_RPi_hat:SPTH_V1,5" H 8000 3800 50  0001 C CNN
 F 3 "~" H 8000 3800 50  0001 C CNN
 	1    8000 3800
@@
 	1    0    0    -1
 $EndComp
+$Comp
+L Morfeas_Rpi_Hat:TLV70433DBVT U3
+U 1 1 5E056599
+P 3600 1050
+F 0 "U3" H 3300 1350 60  0000 L CNN
+F 1 "TLV70433" H 3300 1250 60  0000 L CNN
+F 2 "Morfeas_RPi_hat:TLV70433DBVT" H 4100 900 60  0001 C CNN
+F 3 "" H 3000 1300 60  0000 C CNN
+	1    3600 1050
+	1    0    0    -1
+$EndComp
+$Comp
+L Connector:Conn_01x03_Male J5
+U 1 1 5E075351
+P 6400 5150
+F 0 "J5" H 6372 5174 50  0000 R CNN
+F 1 "RS_232" H 6372 5083 50  0000 R CNN
+F 2 "Connectors_Molex:Molex_KK-6410-03_03x2.54mm_Straight" H 6400 5150 50  0001 C CNN
+F 3 "~" H 6400 5150 50  0001 C CNN
+	1    6400 5150
+	-1   0    0    -1
+$EndComp
+Wire Wire Line
+	5800 4850 6000 4850
+Wire Wire Line
+	6000 4850 6000 5050
+Wire Wire Line
+	6000 5050 6200 5050
+Wire Wire Line
+	5800 5150 6200 5150
+Wire Wire Line
+	6200 5250 6000 5250
+Wire Wire Line
+	6000 5250 6000 5350
+$Comp
+L power:GND #PWR044
+U 1 1 5E093460
+P 6000 5350
+F 0 "#PWR044" H 6000 5100 50  0001 C CNN
+F 1 "GND" H 6005 5177 50  0000 C CNN
+F 2 "" H 6000 5350 50  0001 C CNN
+F 3 "" H 6000 5350 50  0001 C CNN
+	1    6000 5350
+	1    0    0    -1
+$EndComp

Commit message: Update
Parts:
- BT1: footprint Battery:BatteryHolder_Keystone_103_1x20mm -> Morfeas_RPi_hat:CH252032LF
Changed lines of the file:
@@
 F 0 "BT1" H 3568 6696 50  0000 L CNN
 F 1 "Battery_Cell" H 3568 6605 50  0000 L CNN
-F 2 "Battery:BatteryHolder_Keystone_103_1x20mm" V 3450 6660 50  0001 C CNN
+F 2 "Morfeas_RPi_hat:CH252032LF" V 3450 6660 50  0001 C CNN
 F 3 "~" V 3450 6660 50  0001 C CNN
 	1    3450 6600

Commit message: Update
Other:
- note added: "Configuration EEPROM"
- moved on the sheet: C8, U5
Changed lines of the file:
@@
 L Morfeas_Rpi_Hat:24AA08T-I_OT U5
 U 1 1 5E05839E
-P 5550 2950
-F 0 "U5" H 5200 3300 60  0000 L CNN
-F 1 "24AA08" H 5600 2600 60  0000 L CNN
-F 2 "Morfeas_RPi_Hat:24AA08T-I&slash_OT" H 5900 2450 60  0001 C CNN
-F 3 "" H 4900 3700 60  0000 C CNN
-	1    5550 2950
+P 6200 1300
+F 0 "U5" H 5850 1650 60  0000 L CNN
+F 1 "24AA08" H 6250 950 60  0000 L CNN
+F 2 "Morfeas_RPi_Hat:24AA08T-I&slash_OT" H 6550 800 60  0001 C CNN
+F 3 "" H 5550 2050 60  0000 C CNN
+	1    6200 1300
 	1    0    0    -1
 $EndComp
@@
 L power:GND #PWR027
 U 1 1 5E059341
-P 5550 3350
-F 0 "#PWR027" H 5550 3100 50  0001 C CNN
-F 1 "GND" H 5555 3177 50  0000 C CNN
-F 2 "" H 5550 3350 50  0001 C CNN
-F 3 "" H 5550 3350 50  0001 C CNN
-	1    5550 3350
+P 6200 1700
+F 0 "#PWR027" H 6200 1450 50  0001 C CNN
+F 1 "GND" H 6205 1527 50  0000 C CNN
+F 2 "" H 6200 1700 50  0001 C CNN
+F 3 "" H 6200 1700 50  0001 C CNN
+	1    6200 1700
 	1    0    0    -1
 $EndComp
@@
 	8750 1150 8800 1150
 Wire Wire Line
-	6000 2950 6050 2950
-Wire Wire Line
-	6050 2950 6050 3000
+	6650 1300 6700 1300
+Wire Wire Line
+	6700 1300 6700 1350
 Text GLabel 8300 2050 0    50   Input ~ 0
 SDA
-Text GLabel 5000 3000 0    50   Input ~ 0
+Text GLabel 5650 1350 0    50   Input ~ 0
 SCL
 Wire Wire Line
-	5000 3000 5100 3000
-Wire Wire Line
-	5000 2850 5100 2850
+	5650 1350 5750 1350
+Wire Wire Line
+	5650 1200 5750 1200
 Connection ~ 9150 1150
 Wire Wire Line
@@
 Text GLabel 8300 2150 0    50   Input ~ 0
 SCL
-Text GLabel 5000 2850 0    50   Input ~ 0
+Text GLabel 5650 1200 0    50   Input ~ 0
 SDA
 $Comp
@@
 L power:+3.3V #PWR026
 U 1 1 5E059A1A
-P 5550 2450
-F 0 "#PWR026" H 5550 2300 50  0001 C CNN
-F 1 "+3.3V" H 5565 2623 50  0000 C CNN
-F 2 "" H 5550 2450 50  0001 C CNN
-F 3 "" H 5550 2450 50  0001 C CNN
-	1    5550 2450
-	1    0    0    -1
-$EndComp
-Wire Wire Line
-	5550 2450 5550 2500
-Wire Wire Line
-	5650 2500 5550 2500
-Connection ~ 5550 2500
-Wire Wire Line
-	5550 2500 5550 2550
+P 6200 800
+F 0 "#PWR026" H 6200 650 50  0001 C CNN
+F 1 "+3.3V" H 6215 973 50  0000 C CNN
+F 2 "" H 6200 800 50  0001 C CNN
+F 3 "" H 6200 800 50  0001 C CNN
+	1    6200 800
+	1    0    0    -1
+$EndComp
+Wire Wire Line
+	6200 800  6200 850
+Wire Wire Line
+	6300 850  6200 850
+Connection ~ 6200 850
+Wire Wire Line
+	6200 850  6200 900
 $Comp
 L Device:C_Small C8
 U 1 1 5E09628B
-P 5750 2500
-F 0 "C8" V 5650 2500 50  0000 C CNN
-F 1 "100nf" V 5850 2500 50  0000 C CNN
-F 2 "Capacitor_SMD:C_0805_2012Metric" H 5750 2500 50  0001 C CNN
-F 3 "~" H 5750 2500 50  0001 C CNN
-	1    5750 2500
+P 6400 850
+F 0 "C8" V 6300 850 50  0000 C CNN
+F 1 "100nf" V 6500 850 50  0000 C CNN
+F 2 "Capacitor_SMD:C_0805_2012Metric" H 6400 850 50  0001 C CNN
+F 3 "~" H 6400 850 50  0001 C CNN
+	1    6400 850
 	0    1    1    0
 $EndComp
@@
 L power:GND #PWR031
 U 1 1 5E0769C0
-P 6050 3000
-F 0 "#PWR031" H 6050 2750 50  0001 C CNN
-F 1 "GND" H 6055 2827 50  0000 C CNN
-F 2 "" H 6050 3000 50  0001 C CNN
-F 3 "" H 6050 3000 50  0001 C CNN
-	1    6050 3000
+P 6700 1350
+F 0 "#PWR031" H 6700 1100 50  0001 C CNN
+F 1 "GND" H 6705 1177 50  0000 C CNN
+F 2 "" H 6700 1350 50  0001 C CNN
+F 3 "" H 6700 1350 50  0001 C CNN
+	1    6700 1350
 	1    0    0    -1
 $EndComp
@@
 L power:GND #PWR028
 U 1 1 5E097593
-P 5850 2500
-F 0 "#PWR028" H 5850 2250 50  0001 C CNN
-F 1 "GND" H 5855 2327 50  0000 C CNN
-F 2 "" H 5850 2500 50  0001 C CNN
-F 3 "" H 5850 2500 50  0001 C CNN
-	1    5850 2500
+P 6500 850
+F 0 "#PWR028" H 6500 600 50  0001 C CNN
+F 1 "GND" H 6505 677 50  0000 C CNN
+F 2 "" H 6500 850 50  0001 C CNN
+F 3 "" H 6500 850 50  0001 C CNN
+	1    6500 850
 	0    -1   -1   0
 $EndComp
@@
 	1    0    0    -1
 $EndComp
+Wire Notes Line width 20 style dash_dot rgb(255, 0, 0)
+	5200 550  7050 550
+Wire Notes Line width 20 style dash_dot rgb(255, 0, 0)
+	7050 550  7050 2200
+Wire Notes Line width 20 style dash_dot rgb(255, 0, 0)
+	6950 2200 5200 2200
+Wire Notes Line width 20 style dash_dot rgb(255, 0, 0)
+	5200 2200 5200 550
+Text Notes 5250 2150 0    100  ~ 20
+Configuration EEPROM
+Wire Notes Line width 20 style dash_dot rgb(255, 0, 0)
+	7000 1950 5200 1950
 $EndSCHEMATC
