File: src/Morfeas_RPi_Hat/Hardware/Morfeas_Rpi_Hat.sch (KiCad schematic (older format))
At the start: 53 parts, among them J1 Power IN, J2 RPi_header, J3 CAN0_Power+, J4 CAN1_Power+, J5 RS_232, Q1 SUM110P06, Q2 SUM110P06, U1 DS3231, U2 TSR2-2450, U3 TLV70433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

Commit message: Update
Parts:
- added D? (x2): D_ALT, symbol Device:D_ALT
- C15: footprint Capacitors_SMD:C_0805 -> Capacitor_SMD:C_0805_2012Metric
- D1: footprint Diodes_ThroughHole:D_DO-41_SOD81_P10.16mm_Horizontal -> Diode_THT:D_DO-41_SOD81_P10.16mm_Horizontal
- D4: footprint Pin_Headers:Pin_Header_Straight_1x04_Pitch2.54mm -> Connector_PinHeader_2.54mm:PinHeader_1x04_P2.54mm_Vertical
- J5: footprint Pin_Headers:Pin_Header_Straight_1x03_Pitch2.54mm -> Connector_PinHeader_2.54mm:PinHeader_1x03_P2.54mm_Vertical
- R12, R13: footprint Resistors_SMD:R_1206 -> Resistor_SMD:R_1206_3216Metric
Connections:
- net GND: now also D?.2 (A), D?.2 (A)
- net at J3.1 (Pin_1), J3.2 (Pin_2), J3.3 (Pin_3)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: now also D?.1 (K)
- net at J4.1 (Pin_1), J4.2 (Pin_2), J4.3 (Pin_3)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: now also D?.1 (K)
Changed lines of the file:
@@
 	8300 1250 8300 1150
 Wire Wire Line
-	8750 1150 8300 1150
+	8750 1150 8400 1150
 Connection ~ 8750 1150
 Text GLabel 8300 2150 0    50   Input ~ 0
@@
 F 0 "D1" H 1346 921 50  0000 R CNN
 F 1 "1N4007" H 1450 1100 50  0000 R CNN
-F 2 "Diodes_ThroughHole:D_DO-41_SOD81_P10.16mm_Horizontal" H 1300 1000 50  0001 C CNN
+F 2 "Diode_THT:D_DO-41_SOD81_P10.16mm_Horizontal" H 1300 1000 50  0001 C CNN
 F 3 "~" H 1300 1000 50  0001 C CNN
 	1    1300 1000
@@
 Wire Wire Line
 	9950 3800 9150 3800
-Wire Wire Line
-	8200 3700 8300 3700
-Wire Wire Line
-	8300 3700 8300 3800
-Wire Wire Line
-	8300 3800 8200 3800
-Wire Wire Line
-	8200 3900 8300 3900
 Connection ~ 8300 3800
-Wire Wire Line
-	8300 3900 8300 3800
-Wire Wire Line
-	8750 3800 8300 3800
 Connection ~ 8750 3800
 Text GLabel 8300 4800 0    50   Input ~ 0
@@
 NoConn ~ 2450 4400
 $Comp
-L Connector:Conn_01x03_Female J4
-U 1 1 5E14E7A3
-P 8000 3800
-F 0 "J4" H 7892 4085 50  0000 C CNN
-F 1 "CAN1_Power+" H 7892 3994 50  0000 C CNN
-F 2 "Morfeas_RPi_hat:SPTH_V1,5" H 8000 3800 50  0001 C CNN
-F 3 "~" H 8000 3800 50  0001 C CNN
-	1    8000 3800
-	-1   0    0    -1
-$EndComp
-$Comp
 L Mechanical:MountingHole H1
 U 1 1 5E2EEC57
@@
 F 0 "J5" H 7072 3924 50  0000 R CNN
 F 1 "RS_232" H 7072 3833 50  0000 R CNN
-F 2 "Pin_Headers:Pin_Header_Straight_1x03_Pitch2.54mm" H 7100 3900 50  0001 C CNN
+F 2 "Connector_PinHeader_2.54mm:PinHeader_1x03_P2.54mm_Vertical" H 7100 3900 50  0001 C CNN
 F 3 "~" H 7100 3900 50  0001 C CNN
 	1    7100 3900
@@
 F 0 "D4" H 2200 6297 50  0000 C CNN
 F 1 "Status_LEDs" H 2200 6206 50  0000 C CNN
-F 2 "Pin_Headers:Pin_Header_Straight_1x04_Pitch2.54mm" H 2200 5750 50  0001 C CNN
+F 2 "Connector_PinHeader_2.54mm:PinHeader_1x04_P2.54mm_Vertical" H 2200 5750 50  0001 C CNN
 F 3 "~" H 2200 5750 50  0001 C CNN
 	1    2200 5800
@@
 F 0 "C15" V 6650 5400 50  0000 C CNN
 F 1 "100nf" V 6850 5400 50  0000 C CNN
-F 2 "Capacitors_SMD:C_0805" H 6750 5400 50  0001 C CNN
+F 2 "Capacitor_SMD:C_0805_2012Metric" H 6750 5400 50  0001 C CNN
 F 3 "~" H 6750 5400 50  0001 C CNN
 	1    6750 5400
@@
 F 0 "R12" H 1650 2800 50  0000 C CNN
 F 1 "1kΩ" V 1650 3000 50  0000 C CNN
-F 2 "Resistors_SMD:R_1206" V 1590 2940 50  0001 C CNN
+F 2 "Resistor_SMD:R_1206_3216Metric" V 1590 2940 50  0001 C CNN
 F 3 "~" H 1550 2950 50  0001 C CNN
 	1    1550 2950
@@
 F 0 "R13" H 1850 2800 50  0000 C CNN
 F 1 "1kΩ" V 1850 3000 50  0000 C CNN
-F 2 "Resistors_SMD:R_1206" V 1790 2940 50  0001 C CNN
+F 2 "Resistor_SMD:R_1206_3216Metric" V 1790 2940 50  0001 C CNN
 F 3 "~" H 1750 2950 50  0001 C CNN
 	1    1750 2950
@@
 NoConn ~ 2450 3600
 NoConn ~ 1950 3400
+Wire Wire Line
+	8300 3700 8300 3800
+Wire Wire Line
+	8200 3900 8300 3900
+Wire Wire Line
+	8300 3800 8200 3800
+Wire Wire Line
+	8200 3700 8300 3700
+$Comp
+L Connector:Conn_01x03_Female J4
+U 1 1 5E14E7A3
+P 8000 3800
+F 0 "J4" H 7892 4085 50  0000 C CNN
+F 1 "CAN1_Power+" H 7892 3994 50  0000 C CNN
+F 2 "Morfeas_RPi_hat:SPTH_V1,5" H 8000 3800 50  0001 C CNN
+F 3 "~" H 8000 3800 50  0001 C CNN
+	1    8000 3800
+	-1   0    0    -1
+$EndComp
+Wire Wire Line
+	8300 3900 8300 3800
+Wire Wire Line
+	8750 3800 8400 3800
+$Comp
+L Device:D_ALT D?
+U 1 1 5E0B78DF
+P 8600 3450
+F 0 "D?" V 8500 3550 50  0000 R CNN
+F 1 "D_ALT" H 8700 3350 50  0000 R CNN
+F 2 "" H 8600 3450 50  0001 C CNN
+F 3 "~" H 8600 3450 50  0001 C CNN
+	1    8600 3450
+	1    0    0    1
+$EndComp
+$Comp
+L power:GND #PWR?
+U 1 1 5E12E002
+P 8750 3500
+F 0 "#PWR?" H 8750 3250 50  0001 C CNN
+F 1 "GND" H 8755 3327 50  0000 C CNN
+F 2 "" H 8750 3500 50  0001 C CNN
+F 3 "" H 8750 3500 50  0001 C CNN
+	1    8750 3500
+	1    0    0    -1
+$EndComp
+Wire Wire Line
+	8750 3450 8750 3500
+Wire Wire Line
+	8450 3450 8400 3450
+Wire Wire Line
+	8400 3450 8400 3800
+Connection ~ 8400 3800
+Wire Wire Line
+	8400 3800 8300 3800
+$Comp
+L Device:D_ALT D?
+U 1 1 5E165919
+P 8600 800
+F 0 "D?" V 8500 900 50  0000 R CNN
+F 1 "D_ALT" H 8700 700 50  0000 R CNN
+F 2 "" H 8600 800 50  0001 C CNN
+F 3 "~" H 8600 800 50  0001 C CNN
+	1    8600 800
+	1    0    0    1
+$EndComp
+$Comp
+L power:GND #PWR?
+U 1 1 5E16591F
+P 8750 850
+F 0 "#PWR?" H 8750 600 50  0001 C CNN
+F 1 "GND" H 8755 677 50  0000 C CNN
+F 2 "" H 8750 850 50  0001 C CNN
+F 3 "" H 8750 850 50  0001 C CNN
+	1    8750 850
+	1    0    0    -1
+$EndComp
+Wire Wire Line
+	8750 800  8750 850
+Wire Wire Line
+	8450 800  8400 800
+Wire Wire Line
+	8400 800  8400 1150
+Connection ~ 8400 1150
+Wire Wire Line
+	8400 1150 8300 1150
 $EndSCHEMATC

Commit message: Update Morfeas_RPi_Hat
Parts:
- D5, D6: renamed from D?; value D_ALT -> NRVTSA4100ET3G; footprint (none) -> Morfeas_RPi_hat:DO-214AC(SMA)
Changed lines of the file:
@@
 	8750 3800 8400 3800
 $Comp
-L Device:D_ALT D?
+L Device:D_ALT D6
 U 1 1 5E0B78DF
 P 8600 3450
-F 0 "D?" V 8500 3550 50  0000 R CNN
-F 1 "D_ALT" H 8700 3350 50  0000 R CNN
-F 2 "" H 8600 3450 50  0001 C CNN
+F 0 "D6" H 8550 3500 50  0000 R CNN
+F 1 "NRVTSA4100ET3G" H 8700 3350 50  0000 R CNN
+F 2 "Morfeas_RPi_hat:DO-214AC(SMA)" H 8600 3450 50  0001 C CNN
 F 3 "~" H 8600 3450 50  0001 C CNN
 	1    8600 3450
@@
 $EndComp
 $Comp
-L power:GND #PWR?
+L power:GND #PWR048
 U 1 1 5E12E002
 P 8750 3500
-F 0 "#PWR?" H 8750 3250 50  0001 C CNN
+F 0 "#PWR048" H 8750 3250 50  0001 C CNN
 F 1 "GND" H 8755 3327 50  0000 C CNN
 F 2 "" H 8750 3500 50  0001 C CNN
@@
 	8400 3800 8300 3800
 $Comp
-L Device:D_ALT D?
+L Device:D_ALT D5
 U 1 1 5E165919
 P 8600 800
-F 0 "D?" V 8500 900 50  0000 R CNN
-F 1 "D_ALT" H 8700 700 50  0000 R CNN
-F 2 "" H 8600 800 50  0001 C CNN
+F 0 "D5" H 8550 850 50  0000 R CNN
+F 1 "NRVTSA4100ET3G" H 8700 700 50  0000 R CNN
+F 2 "Morfeas_RPi_hat:DO-214AC(SMA)" H 8600 800 50  0001 C CNN
 F 3 "~" H 8600 800 50  0001 C CNN
 	1    8600 800
@@
 $EndComp
 $Comp
-L power:GND #PWR?
+L power:GND #PWR047
 U 1 1 5E16591F
 P 8750 850
-F 0 "#PWR?" H 8750 600 50  0001 C CNN
+F 0 "#PWR047" H 8750 600 50  0001 C CNN
 F 1 "GND" H 8755 677 50  0000 C CNN
 F 2 "" H 8750 850 50  0001 C CNN

Commit message: Update Morfeas_RPi_Hat
Parts:
- removed J1: Power IN, Morfeas_RPi_hat:SPTH_V1,5, symbol Connector:Conn_01x03_Female
- removed J3: CAN0_Power+, Morfeas_RPi_hat:SPTH_V1,5, symbol Connector:Conn_01x03_Female
- removed J4: CAN1_Power+, Morfeas_RPi_hat:SPTH_V1,5, symbol Connector:Conn_01x03_Female
- added J1: Con, Morfeas_RPi_hat:SPT1.5_8-H-3.5, symbol Morfeas_Rpi_Hat:Connector
Connections:
- net +24V: now also J1.5
- net GND: now also J1.2, J1.3, J1.4, J1.6, J1.8
- net at D5.1 (K), R1.2, U6.3 (RS-): now also J1.7
- net at D6.1 (K), R2.2, U7.3 (RS-): now also J1.1
Other:
- moved on the sheet: H1, H2, H3, H4
Changed lines of the file:
@@
 Wire Wire Line
 	9950 1150 9150 1150
-$Comp
-L Connector:Conn_01x03_Female J3
-U 1 1 5E088EC8
-P 8000 1150
-F 0 "J3" H 7892 1435 50  0000 C CNN
-F 1 "CAN0_Power+" H 7892 1344 50  0000 C CNN
-F 2 "Morfeas_RPi_hat:SPTH_V1,5" H 8000 1150 50  0001 C CNN
-F 3 "~" H 8000 1150 50  0001 C CNN
-	1    8000 1150
-	-1   0    0    -1
-$EndComp
-Wire Wire Line
-	8200 1050 8300 1050
-Wire Wire Line
-	8300 1050 8300 1150
-Wire Wire Line
-	8300 1150 8200 1150
-Wire Wire Line
-	8200 1250 8300 1250
-Connection ~ 8300 1150
-Wire Wire Line
-	8300 1250 8300 1150
 Wire Wire Line
 	8750 1150 8400 1150
@@
 Wire Wire Line
 	9950 3800 9150 3800
-Connection ~ 8300 3800
 Connection ~ 8750 3800
 Text GLabel 8300 4800 0    50   Input ~ 0
@@
 Text Notes 590  1760 0    100  ~ 20
 Power Supply Unit
-$Comp
-L Connector:Conn_01x03_Female J1
-U 1 1 5E179F8A
-P 800 1100
-F 0 "J1" H 750 1300 50  0000 C CNN
-F 1 "Power IN" V 900 1100 50  0000 C CNN
-F 2 "Morfeas_RPi_hat:SPTH_V1,5" H 800 1100 50  0001 C CNN
-F 3 "~" H 800 1100 50  0001 C CNN
-	1    800  1100
-	-1   0    0    -1
-$EndComp
 Wire Notes Line width 20 style dash_dot rgb(255, 0, 0)
 	4500 550  4500 1800
@@
 	1000 1000 1100 1000
 Connection ~ 1100 1000
-Wire Wire Line
-	1000 1100 1100 1100
-Wire Wire Line
-	1100 1100 1100 1000
 Wire Wire Line
 	1150 1000 1100 1000
@@
 L Mechanical:MountingHole H1
 U 1 1 5E2EEC57
-P 8650 6000
-F 0 "H1" H 8750 6046 50  0000 L CNN
-F 1 "MountingHole" H 8750 5955 50  0000 L CNN
-F 2 "MountingHole:MountingHole_3mm" H 8650 6000 50  0001 C CNN
-F 3 "~" H 8650 6000 50  0001 C CNN
-	1    8650 6000
+P 9750 6000
+F 0 "H1" H 9850 6046 50  0000 L CNN
+F 1 "MountingHole" H 9850 5955 50  0000 L CNN
+F 2 "MountingHole:MountingHole_3mm" H 9750 6000 50  0001 C CNN
+F 3 "~" H 9750 6000 50  0001 C CNN
+	1    9750 6000
 	1    0    0    -1
 $EndComp
@@
 L Mechanical:MountingHole H2
 U 1 1 5E2F00AC
-P 8650 6200
-F 0 "H2" H 8750 6246 50  0000 L CNN
-F 1 "MountingHole" H 8750 6155 50  0000 L CNN
-F 2 "MountingHole:MountingHole_3mm" H 8650 6200 50  0001 C CNN
-F 3 "~" H 8650 6200 50  0001 C CNN
-	1    8650 6200
+P 9750 6200
+F 0 "H2" H 9850 6246 50  0000 L CNN
+F 1 "MountingHole" H 9850 6155 50  0000 L CNN
+F 2 "MountingHole:MountingHole_3mm" H 9750 6200 50  0001 C CNN
+F 3 "~" H 9750 6200 50  0001 C CNN
+	1    9750 6200
 	1    0    0    -1
 $EndComp
@@
 L Mechanical:MountingHole H3
 U 1 1 5E2F0330
-P 9450 6000
-F 0 "H3" H 9550 6046 50  0000 L CNN
-F 1 "MountingHole" H 9550 5955 50  0000 L CNN
-F 2 "MountingHole:MountingHole_3mm" H 9450 6000 50  0001 C CNN
-F 3 "~" H 9450 6000 50  0001 C CNN
-	1    9450 6000
+P 10550 6000
+F 0 "H3" H 10650 6046 50  0000 L CNN
+F 1 "MountingHole" H 10650 5955 50  0000 L CNN
+F 2 "MountingHole:MountingHole_3mm" H 10550 6000 50  0001 C CNN
+F 3 "~" H 10550 6000 50  0001 C CNN
+	1    10550 6000
 	1    0    0    -1
 $EndComp
@@
 L Mechanical:MountingHole H4
 U 1 1 5E2F07C8
-P 9450 6200
-F 0 "H4" H 9550 6246 50  0000 L CNN
-F 1 "MountingHole" H 9550 6155 50  0000 L CNN
-F 2 "MountingHole:MountingHole_3mm" H 9450 6200 50  0001 C CNN
-F 3 "~" H 9450 6200 50  0001 C CNN
-	1    9450 6200
+P 10550 6200
+F 0 "H4" H 10650 6246 50  0000 L CNN
+F 1 "MountingHole" H 10650 6155 50  0000 L CNN
+F 2 "MountingHole:MountingHole_3mm" H 10550 6200 50  0001 C CNN
+F 3 "~" H 10550 6200 50  0001 C CNN
+	1    10550 6200
 	1    0    0    -1
 $EndComp
@@
 NoConn ~ 1950 3400
 Wire Wire Line
-	8300 3700 8300 3800
-Wire Wire Line
-	8200 3900 8300 3900
-Wire Wire Line
-	8300 3800 8200 3800
-Wire Wire Line
-	8200 3700 8300 3700
-$Comp
-L Connector:Conn_01x03_Female J4
-U 1 1 5E14E7A3
-P 8000 3800
-F 0 "J4" H 7892 4085 50  0000 C CNN
-F 1 "CAN1_Power+" H 7892 3994 50  0000 C CNN
-F 2 "Morfeas_RPi_hat:SPTH_V1,5" H 8000 3800 50  0001 C CNN
-F 3 "~" H 8000 3800 50  0001 C CNN
-	1    8000 3800
-	-1   0    0    -1
-$EndComp
-Wire Wire Line
-	8300 3900 8300 3800
-Wire Wire Line
 	8750 3800 8400 3800
 $Comp
@@
 	8400 3450 8400 3800
 Connection ~ 8400 3800
-Wire Wire Line
-	8400 3800 8300 3800
 $Comp
 L Device:D_ALT D5
@@
 	8400 800  8400 1150
 Connection ~ 8400 1150
-Wire Wire Line
-	8400 1150 8300 1150
+$Comp
+L Morfeas_Rpi_Hat:Connector J1
+U 7 1 5E1162EB
+P 8000 1150
+F 0 "J1" H 7892 965 50  0000 C CNN
+F 1 "Con" H 7892 1056 50  0001 C CNN
+F 2 "Morfeas_RPi_hat:SPT1.5_8-H-3.5" H 8000 1150 50  0001 C CNN
+F 3 "" H 8000 1150 50  0001 C CNN
+	7    8000 1150
+	-1   0    0    1
+$EndComp
+Wire Wire Line
+	8200 1150 8400 1150
+Wire Wire Line
+	8250 1400 8400 1400
+Wire Wire Line
+	8400 1400 8400 1500
+$Comp
+L power:GND #PWR049
+U 1 1 5E15111B
+P 8400 1500
+F 0 "#PWR049" H 8400 1250 50  0001 C CNN
+F 1 "GND" H 8250 1450 50  0000 C CNN
+F 2 "" H 8400 1500 50  0001 C CNN
+F 3 "" H 8400 1500 50  0001 C CNN
+	1    8400 1500
+	1    0    0    -1
+$EndComp
+Wire Wire Line
+	8200 3800 8400 3800
+$Comp
+L Morfeas_Rpi_Hat:Connector J1
+U 1 1 5E16FE86
+P 8000 3800
+F 0 "J1" H 7892 3615 50  0000 C CNN
+F 1 "Con" H 7892 3706 50  0000 C CNN
+F 2 "Morfeas_RPi_hat:SPT1.5_8-H-3.5" H 8000 3800 50  0001 C CNN
+F 3 "" H 8000 3800 50  0001 C CNN
+	1    8000 3800
+	-1   0    0    1
+$EndComp
+$Comp
+L Morfeas_Rpi_Hat:Connector J1
+U 5 1 5E171471
+P 800 1000
+F 0 "J1" H 650 900 50  0000 C CNN
+F 1 "Con" H 900 1000 50  0001 C CNN
+F 2 "Morfeas_RPi_hat:SPT1.5_8-H-3.5" H 800 1000 50  0001 C CNN
+F 3 "" H 800 1000 50  0001 C CNN
+	5    800  1000
+	-1   0    0    1
+$EndComp
+$Comp
+L Morfeas_Rpi_Hat:Connector J1
+U 6 1 5E172C37
+P 800 1200
+F 0 "J1" H 650 1100 50  0000 C CNN
+F 1 "Con" H 900 1200 50  0001 C CNN
+F 2 "Morfeas_RPi_hat:SPT1.5_8-H-3.5" H 800 1200 50  0001 C CNN
+F 3 "" H 800 1200 50  0001 C CNN
+	6    800  1200
+	-1   0    0    1
+$EndComp
+$Comp
+L power:GND #PWR0106
+U 1 1 5E1939E0
+P 8400 6250
+F 0 "#PWR0106" H 8400 6000 50  0001 C CNN
+F 1 "GND" H 8405 6077 50  0000 C CNN
+F 2 "" H 8400 6250 50  0001 C CNN
+F 3 "" H 8400 6250 50  0001 C CNN
+	1    8400 6250
+	1    0    0    -1
+$EndComp
+Wire Wire Line
+	8400 6200 8400 6250
+Wire Wire Line
+	8400 6200 8400 6100
+Connection ~ 8400 6200
+Connection ~ 8400 6000
+Wire Wire Line
+	8400 6000 8400 5900
+Connection ~ 8400 6100
+Wire Wire Line
+	8400 6100 8400 6000
+Wire Wire Line
+	8300 6200 8400 6200
+Wire Wire Line
+	8300 6100 8400 6100
+Wire Wire Line
+	8300 6000 8400 6000
+Wire Wire Line
+	8400 5900 8300 5900
+$Comp
+L Morfeas_Rpi_Hat:Connector J1
+U 8 1 5E1755AF
+P 8100 5900
+F 0 "J1" H 8150 5900 50  0000 L CNN
+F 1 "Con" V 8150 5700 50  0001 L CNN
+F 2 "Morfeas_RPi_hat:SPT1.5_8-H-3.5" H 8100 5900 50  0001 C CNN
+F 3 "" H 8100 5900 50  0001 C CNN
+	8    8100 5900
+	-1   0    0    -1
+$EndComp
+$Comp
+L Morfeas_Rpi_Hat:Connector J1
+U 4 1 5E174B4D
+P 8100 6000
+F 0 "J1" H 8150 6000 50  0000 L CNN
+F 1 "Con" V 8150 5800 50  0001 L CNN
+F 2 "Morfeas_RPi_hat:SPT1.5_8-H-3.5" H 8100 6000 50  0001 C CNN
+F 3 "" H 8100 6000 50  0001 C CNN
+	4    8100 6000
+	-1   0    0    -1
+$EndComp
+$Comp
+L Morfeas_Rpi_Hat:Connector J1
+U 3 1 5E1737B5
+P 8100 6100
+F 0 "J1" H 8150 6100 50  0000 L CNN
+F 1 "Con" V 8150 5900 50  0001 L CNN
+F 2 "Morfeas_RPi_hat:SPT1.5_8-H-3.5" H 8100 6100 50  0001 C CNN
+F 3 "" H 8100 6100 50  0001 C CNN
+	3    8100 6100
+	-1   0    0    -1
+$EndComp
+$Comp
+L Morfeas_Rpi_Hat:Connector J1
+U 2 1 5E12235A
+P 8100 6200
+F 0 "J1" H 8150 6200 50  0000 L CNN
+F 1 "Con" V 8150 6000 50  0001 L CNN
+F 2 "Morfeas_RPi_hat:SPT1.5_8-H-3.5" H 8100 6200 50  0001 C CNN
+F 3 "" H 8100 6200 50  0001 C CNN
+	2    8100 6200
+	-1   0    0    -1
+$EndComp
 $EndSCHEMATC

Commit message: Update Morfeas_RPi_Hat
Parts:
- D1: footprint Diode_THT:D_DO-41_SOD81_P10.16mm_Horizontal -> Morfeas_RPi_hat:DO-214AC(SMA)
- L1: footprint Inductor_THT:L_Axial_L6.6mm_D2.7mm_P10.16mm_Horizontal_Vishay_IM-2 -> Resistors_SMD:R_2816_HandSoldering
Other:
- note added: "RPi Header"
- moved on the sheet: BT1, C1, C10, C11, C12, C13, C14, C15, C2, C3, C4, C5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

Commit message: Update Morfeas_RPi_Hat files
Parts:
- added C16, C17: 100nf, Capacitor_SMD:C_0805_2012Metric, symbol Device:C_Small
- added R14, R15: 2.2kΩ, Resistor_SMD:R_1206_3216Metric, symbol Device:R_US
- D5, D6: footprint Morfeas_RPi_hat:DO-214AC(SMA) -> Morfeas_RPi_Hat:DO-214AC(SMA)
- J1: footprint Morfeas_RPi_hat:SPT1.5_8-H-3.5 -> Morfeas_RPi_Hat:SPT1.5_8-H-3.5
- L1: footprint Resistors_SMD:R_2816_HandSoldering -> Resistor_SMD:R_2816_7142Metric_Pad3.20x4.45mm_HandSolder
Connections:
- net +24V: now also J1.4, R14.2, R15.2; no longer J1.5
- net GND: now also J1.5, J1.7; no longer J1.4, J1.6
- net at U6.1 (OUT): now also R7.2; no longer R7.1
- net CAN0_P+: now reaches D5.1 (K), R1.2, U6.3 (RS-)
- net CAN0_P+: now also J1.6; no longer J1.7
- net at D2.2 (A), Q1.1 (G), R9.1: now also R7.1, C16.1; no longer R7.2
- net CAN1_P+: now reaches D6.1 (K), J1.1, R2.2, U7.3 (RS-)
- net at D3.2 (A), Q2.1 (G), R10.1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: now also C17.1
- new net: C16.2, R14.1
- new net: C17.2, R15.1
Other:
- moved on the sheet: BT1, C1, C10, C11, C12, C13, C14, C15, C2, C3, C4, C5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

Commit message: Update Morfeas_RPi_Hat files
Parts:
- added Morfeas_project_Logo1: Morfeas Project's Logo, Morfeas_RPi_Hat:Morfeas_logo, symbol Morfeas_Rpi_Hat:Morfeas_project_Logo
- H1, H2, H3, H4: footprint MountingHole:MountingHole_3mm -> MountingHole:MountingHole_3.5mm
- J2: symbol Connector_Generic:Conn_02x20_Odd_Even -> Morfeas_Rpi_Hat:Conn_02x20_Odd_Even
- Open_Source_hardware1: footprint Symbols:OSHW-Logo2_7.3x6mm_SilkScreen -> Symbol:OSHW-Logo2_7.3x6mm_SilkScreen
- U2: footprint Morfeas_RPi_hat:TSR2-2450 -> Morfeas_RPi_Hat:TSR2-2450
- U3: footprint Morfeas_RPi_hat:TLV70433DBVT -> Morfeas_RPi_Hat:TLV70433DBVT
Changed lines of the file:
@@
 $EndDescr
 $Comp
-L Connector_Generic:Conn_02x20_Odd_Even J2
+L Morfeas_Rpi_Hat:Conn_02x20_Odd_Even J2
 U 1 1 5E041881
 P 6250 3850
@@
 F 0 "Open_Source_hardware1" H 2250 7275 50  0001 C CNN
 F 1 "Open Source Hardware" H 2250 6775 50  0000 C CNN
-F 2 "Symbols:OSHW-Logo2_7.3x6mm_SilkScreen" H 2250 7000 50  0001 C CNN
+F 2 "Symbol:OSHW-Logo2_7.3x6mm_SilkScreen" H 2250 7000 50  0001 C CNN
 F 3 "~" H 2250 7000 50  0001 C CNN
 	1    2250 7000
@@
 F 0 "U2" H 6000 1200 50  0000 C CNN
 F 1 "TSR2-2450" H 6150 1101 50  0000 C CNN
-F 2 "Morfeas_RPi_hat:TSR2-2450" H 6175 800 50  0001 L CIN
+F 2 "Morfeas_RPi_Hat:TSR2-2450" H 6175 800 50  0001 L CIN
 F 3 "http://www.st.com/content/ccc/resource/technical/document/datasheet/41/4f/b3/b0/12/d4/47/88/CD00000444.pdf/files/CD00000444.pdf/jcr:content/translations/en.CD00000444.pdf" H 6150 900 50  0001 C CNN
 	1    6150 950
@@
 F 0 "H1" H 1100 6646 50  0000 L CNN
 F 1 "MountingHole" H 1100 6555 50  0000 L CNN
-F 2 "MountingHole:MountingHole_3mm" H 1000 6600 50  0001 C CNN
+F 2 "MountingHole:MountingHole_3.5mm" H 1000 6600 50  0001 C CNN
 F 3 "~" H 1000 6600 50  0001 C CNN
 	1    1000 6600
@@
 F 0 "H2" H 1100 6846 50  0000 L CNN
 F 1 "MountingHole" H 1100 6755 50  0000 L CNN
-F 2 "MountingHole:MountingHole_3mm" H 1000 6800 50  0001 C CNN
+F 2 "MountingHole:MountingHole_3.5mm" H 1000 6800 50  0001 C CNN
 F 3 "~" H 1000 6800 50  0001 C CNN
 	1    1000 6800
@@
 F 0 "H3" H 1100 7046 50  0000 L CNN
 F 1 "MountingHole" H 1100 6955 50  0000 L CNN
-F 2 "MountingHole:MountingHole_3mm" H 1000 7000 50  0001 C CNN
+F 2 "MountingHole:MountingHole_3.5mm" H 1000 7000 50  0001 C CNN
 F 3 "~" H 1000 7000 50  0001 C CNN
 	1    1000 7000
@@
 F 0 "H4" H 1100 7246 50  0000 L CNN
 F 1 "MountingHole" H 1100 7155 50  0000 L CNN
-F 2 "MountingHole:MountingHole_3mm" H 1000 7200 50  0001 C CNN
+F 2 "MountingHole:MountingHole_3.5mm" H 1000 7200 50  0001 C CNN
 F 3 "~" H 1000 7200 50  0001 C CNN
 	1    1000 7200
@@
 F 0 "U3" H 6900 1300 60  0000 L CNN
 F 1 "TLV70433" H 6900 1200 60  0000 L CNN
-F 2 "Morfeas_RPi_hat:TLV70433DBVT" H 7700 850 60  0001 C CNN
+F 2 "Morfeas_RPi_Hat:TLV70433DBVT" H 7700 850 60  0001 C CNN
 F 3 "" H 6600 1250 60  0000 C CNN
 	1    7200 1000
@@
 	-1   0    0    1
 $EndComp
+$Comp
+L Morfeas_Rpi_Hat:Morfeas_project_Logo Morfeas_project_Logo1
+U 1 1 5E12A45C
+P 3250 7000
+F 0 "Morfeas_project_Logo1" H 3250 6850 60  0001 C CNN
+F 1 "Morfeas Project's Logo" H 3250 6850 60  0000 C CNN
+F 2 "Morfeas_RPi_Hat:Morfeas_logo" H 3250 7000 75  0001 C CNN
+F 3 "" H 3250 7000 75  0001 C CNN
+	1    3250 7000
+	1    0    0    -1
+$EndComp
 $EndSCHEMATC

Commit message: Update Morfeas_RPi_Hat files
Parts:
- BT1: footprint Morfeas_RPi_hat:CH252032LF -> Morfeas_RPi_Hat:CH252032LF
Changed lines of the file:
@@
 F 0 "BT1" H 10718 3996 50  0000 L CNN
 F 1 "Battery_Cell" H 10718 3905 50  0000 L CNN
-F 2 "Morfeas_RPi_hat:CH252032LF" V 10600 3960 50  0001 C CNN
+F 2 "Morfeas_RPi_Hat:CH252032LF" V 10600 3960 50  0001 C CNN
 F 3 "~" V 10600 3960 50  0001 C CNN
 	1    10600 3900

Commit message: Update Morfeas_RPi_Hat files
Parts:
- J2: footprint Connector_PinSocket_2.54mm:PinSocket_2x20_P2.54mm_Vertical -> Morfeas_RPi_Hat:PinSocket_2x20_P2.54mm_Vertical
Changed lines of the file:
@@
 F 0 "J2" H 6300 4967 50  0000 C CNN
 F 1 "RPi_header" H 6300 4876 50  0000 C CNN
-F 2 "Connector_PinSocket_2.54mm:PinSocket_2x20_P2.54mm_Vertical" H 6250 3850 50  0001 C CNN
+F 2 "Morfeas_RPi_Hat:PinSocket_2x20_P2.54mm_Vertical" H 6250 3850 50  0001 C CNN
 F 3 "~" H 6250 3850 50  0001 C CNN
 	1    6250 3850
