File: src/Morfeas_RPi_Hat/Hardware/Morfeas_Rpi_Hat.kicad_pcb (KiCad board)
At the start: 2 copper layers, 65 x 56 mm, 43 parts, among them J2 RPi_header, Q1 Q_PMOS_GDS, Q2 Q_PMOS_GDS, U1 DS3231, U2 TSR2-2450, U3 TLV70433, U4 SP3232, U5 24AA08, U6 MAX9611, U7 MAX9611

Commit message: Update
Parts:
- BT1: footprint Battery:BatteryHolder_Keystone_106_1x20mm -> Battery:BatteryHolder_Keystone_103_1x20mm
- U1: moved to B.Cu
- moved U1 122.3 mm to (100.5, 89.5), turned to 180 degrees
- moved BT1 79.8 mm to (100.5, 77.5), turned to 270 degrees

Commit message: Update, add some 3d_models
Parts:
- added J1: Power IN, Morfeas_RPi_hat:SPTH_V1,5, F.Cu at (209.5, 51.4)
- added J3: CAN0_Power+, Morfeas_RPi_hat:SPTH_V1,5, F.Cu at (221.7, 51.4)
- added J4: CAN1_Power+, Morfeas_RPi_hat:SPTH_V1,5, F.Cu at (233.8, 51.4)
- U2: footprint Morfeas_RPi_Hat:TSR2-2450 -> Morfeas_RPi_hat:TSR2-2450
- U3: footprint Morfeas_RPi_Hat:24AA08T-I&slash_OT -> Morfeas_RPi_hat:TLV70433DBVT

Commit message: Update
Parts:
- added J5: RS_232, Connectors_Molex:Molex_KK-6410-03_03x2.54mm_Straight, F.Cu at (157.1, 35.9)
Connections:
- U4 pad 13: (no net) -> Net-(J5-Pad2)
- U4 pad 14: (no net) -> Net-(J5-Pad1)

Commit message: Update
Parts:
- BT1: footprint Battery:BatteryHolder_Keystone_103_1x20mm -> Morfeas_RPi_hat:CH252032LF
- Q1, Q2: value Q_PMOS_GDS -> SUM110P06
Changed lines of the file:
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@@
     (add_net +5V)
+  )
+  (module Morfeas_RPi_hat:CH252032LF (layer F.Cu)
+    (at 100.5 77.5 270)
+    (descr CH25-2032LF-1)
+    (tags "Undefined or Miscellaneous")
+    (fp_text reference BT1 (at -5 20) (layer F.SilkS)
+      (effects (font (size 1.27 1.27) (thickness 0.254)))
+    )
+    (fp_text value Battery_Cell (at 0 14.5 90) (layer F.SilkS) hide
+      (effects (font (size 1.27 1.27) (thickness 0.254)))
+    )
+    (fp_line (start -12.4 -6.4) (end 12.4 -6.4) (layer F.CrtYd) (width 0.1))
+    (fp_line (start 12.4 -6.4) (end 12.4 23.4) (layer F.CrtYd) (width 0.1))
+    (fp_line (start 12.4 23.4) (end -12.4 23.4) (layer F.CrtYd) (width 0.1))
+    (fp_line (start -12.4 23.4) (end -12.4 -6.4) (layer F.CrtYd) (width 0.1))
+    (fp_line (start -11.4 6) (end -11.4 6) (layer F.Fab) (width 0.2))
+    (fp_line (start 11.4 6) (end 11.4 6) (layer F.Fab) (width 0.2))
+    (fp_line (start -3.3 16.9) (end -3.3 22.4) (layer F.Fab) (width 0.2))
+    (fp_line (start -3.3 22.4) (end 3.3 22.4) (layer F.Fab) (width 0.2))
+    (fp_line (start 3.3 22.4) (end 3.3 16.9) (layer F.Fab) (width 0.2))
+    (fp_line (start -11.4 6) (end -11.4 6) (layer F.SilkS) (width 0.1))
+    (fp_line (start 11.4 6) (end 11.4 6) (layer F.SilkS) (width 0.1))
+    (fp_line (start -3.3 16.9) (end -3.3 22.4) (layer F.SilkS) (width 0.1))
+    (fp_line (start -3.3 22.4) (end 3.3 22.4) (layer F.SilkS) (width 0.1))
+    (fp_line (start 3.3 22.4) (end 3.3 16.9) (layer F.SilkS) (width 0.1))
+    (fp_arc (start 0 6) (end -11.4 6) (angle -180) (layer F.Fab) (width 0.2))
+    (fp_arc (start 0 6) (end 11.4 6) (angle -180) (layer F.Fab) (width 0.2))
+    (fp_arc (start 0 6) (end -11.4 6) (angle -180) (layer F.SilkS) (width 0.1))
+    (fp_arc (start 0 6) (end 11.4 6) (angle -180) (layer F.SilkS) (width 0.1))
+    (pad 1 thru_hole circle (at 0 0 270) (size 1.65 1.65) (drill 1.1) (layers *.Cu *.Mask)
+      (net 2 "Net-(BT1-Pad1)"))
+    (pad 2 thru_hole circle (at 0 20 270) (size 1.65 1.65) (drill 1.1) (layers *.Cu *.Mask)
+      (net 1 GND))
+    (model ${KIPRJMOD}/Project's_libs/STEP/CH25-2032LF_approx.step
+      (offset (xyz 0 -5.99948 0))
+      (scale (xyz 1 1 1))
+      (rotate (xyz 0 0 180))
+    )
   )
   (module Morfeas_RPi_hat:TLV70433DBVT (layer F.Cu)
@@
       (effects (font (size 1 1) (thickness 0.15)))
     )
-    (fp_text value Q_PMOS_GDS (at 0 6.65) (layer F.Fab)
+    (fp_text value SUM110P06 (at 0 6.65) (layer F.Fab)
       (effects (font (size 1 1) (thickness 0.15)))
     )
@@
       (effects (font (size 1 1) (thickness 0.15)))
     )
-    (fp_text value Q_PMOS_GDS (at 0 6.65) (layer F.Fab)
+    (fp_text value SUM110P06 (at 0 6.65) (layer F.Fab)
       (effects (font (size 1 1) (thickness 0.15)))
     )
@@
       (at (xyz 0 0 0))
       (scale (xyz 1 1 1))
-      (rotate (xyz 0 0 0))
-    )
-  )
-  (module Battery:BatteryHolder_Keystone_103_1x20mm (layer F.Cu)
-    (at 100.5 77.5 270)
-    (descr http://www.keyelco.com/product-pdf.cfm?p=719)
-    (tags "Keystone type 103 battery holder")
-    (fp_text reference BT1 (at 0 -4.3 90) (layer F.SilkS)
-      (effects (font (size 1 1) (thickness 0.15)))
-    )
-    (fp_text value Battery_Cell (at 15 13 90) (layer F.Fab)
-      (effects (font (size 1 1) (thickness 0.15)))
-    )
-    (fp_text user + (at 2.75 0 90) (layer F.SilkS)
-      (effects (font (size 1.5 1.5) (thickness 0.15)))
-    )
-    (fp_text user %R (at 0 0 90) (layer F.Fab)
-      (effects (font (size 1 1) (thickness 0.15)))
-    )
-    (fp_arc (start 15.2 0) (end 4.01 3.6) (angle -162.5) (layer F.CrtYd) (width 0.05))
-    (fp_arc (start 15.2 0) (end 4.01 -3.6) (angle 162.5) (layer F.CrtYd) (width 0.05))
-    (fp_arc (start 3.5 3.8) (end 3.5 3.25) (angle 70) (layer F.CrtYd) (width 0.05))
-    (fp_arc (start 3.5 -3.8) (end 3.5 -3.25) (angle -70) (layer F.CrtYd) (width 0.05))
-    (fp_arc (start 15.2 0) (end 4.25 3.5) (angle -162.5) (layer F.SilkS) (width 0.12))
-    (fp_arc (start 3.5 3.8) (end 3.5 3) (angle 70) (layer F.SilkS) (width 0.12))
-    (fp_arc (start 15.2 0) (end 4.25 -3.5) (angle 162.5) (layer F.SilkS) (width 0.12))
-    (fp_arc (start 3.5 -3.8) (end 3.5 -3) (angle -70) (layer F.SilkS) (width 0.12))
-    (fp_arc (start 3.5 3.8) (end 3.5 2.9) (angle 70) (layer F.Fab) (width 0.1))
-    (fp_arc (start 15.2 0) (end 4.35 3.5) (angle -162.5) (layer F.Fab) (width 0.1))
-    (fp_arc (start 15.2 0) (end 4.35 -3.5) (angle 162.5) (layer F.Fab) (width 0.1))
-    (fp_arc (start 15.2 0) (end 5.2 1.3) (angle -180) (layer F.Fab) (width 0.1))
-    (fp_line (start -2.45 -3.25) (end 3.5 -3.25) (layer F.CrtYd) (width 0.05))
-    (fp_line (start -2.45 3.25) (end 3.5 3.25) (layer F.CrtYd) (width 0.05))
-    (fp_line (start -2.45 3.25) (end -2.45 -3.25) (layer F.CrtYd) (width 0.05))
-    (fp_line (start -2.2 -3) (end 3.5 -3) (layer F.SilkS) (width 0.12))
-    (fp_line (start -2.2 3) (end -2.2 -3) (layer F.SilkS) (width 0.12))
-    (fp_line (start -2.2 3) (end 3.5 3) (layer F.SilkS) (width 0.12))
-    (fp_arc (start 15.2 0) (end 9 1.3) (angle -170) (layer F.Fab) (width 0.1))
-    (fp_arc (start 15.2 0) (end 13.3 1.3) (angle -150) (layer F.Fab) (width 0.1))
-    (fp_line (start 23.5712 7.7216) (end 22.6568 6.8834) (layer F.Fab) (width 0.1))
-    (fp_line (start 23.5712 -7.7216) (end 22.6314 -6.858) (layer F.Fab) (width 0.1))
-    (fp_arc (start 15.2 0) (end 13.3 -1.3) (angle 150) (layer F.Fab) (width 0.1))
-    (fp_arc (start 15.2 0) (end 9 -1.3) (angle 170) (layer F.Fab) (width 0.1))
-    (fp_arc (start 15.2 0) (end 5.2 -1.3) (angle 180) (layer F.Fab) (width 0.1))
-    (fp_line (start 3.5306 -2.9) (end -1.7 -2.9) (layer F.Fab) (width 0.1))
-    (fp_line (start -1.7 2.9) (end 3.5306 2.9) (layer F.Fab) (width 0.1))
-    (fp_line (start -2.1 -2.5) (end -2.1 2.5) (layer F.Fab) (width 0.1))
-    (fp_line (start 0 1.3) (end 16.2 1.3) (layer F.Fab) (width 0.1))
-    (fp_line (start 16.2 -1.3) (end 0 -1.3) (layer F.Fab) (width 0.1))
-    (fp_arc (start 3.5 -3.8) (end 3.5 -2.9) (angle -70) (layer F.Fab) (width 0.1))
-    (fp_arc (start 16.2 0) (end 16.2 -1.3) (angle 180) (layer F.Fab) (width 0.1))
-    (fp_line (start 0 -1.3) (end 0 1.3) (layer F.Fab) (width 0.1))
-    (fp_arc (start -1.7 2.5) (end -2.1 2.5) (angle -90) (layer F.Fab) (width 0.1))
-    (fp_arc (start -1.7 -2.5) (end -2.1 -2.5) (angle 90) (layer F.Fab) (width 0.1))
-    (pad 2 thru_hole circle (at 20.49 0 270) (size 3 3) (drill 1.5) (layers *.Cu *.Mask)
-      (net 1 GND))
-    (pad 1 thru_hole rect (at 0 0 270) (size 3 3) (drill 1.5) (layers *.Cu *.Mask)
-      (net 2 "Net-(BT1-Pad1)"))
-    (model ${KISYS3DMOD}/Battery.3dshapes/BatteryHolder_Keystone_103_1x20mm.wrl
-      (at (xyz 0 0 0))
-      (scale (xyz 1 1 1))

Commit message: Update
Parts:
- added D4: Status_LEDs, LEDs:LED_D5.0mm-4, F.Cu at (130.9, 32.5)
- added R11: 330Ω, Resistors_SMD:R_1206, F.Cu at (139.3, 30.3)
Changed lines of the file:
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@@
     (tracks 0)
     (zones 0)
-    (modules 47)
-    (nets 30)
+    (modules 49)
+    (nets 31)
   )
   (page A4)
@@
   (net 28 "Net-(J5-Pad2)")
   (net 29 "Net-(J5-Pad1)")
+  (net 30 "Net-(D4-Pad1)")
   (net_class Default "This is the default net class."
     (clearance 0.2286)
@@
     (add_net "Net-(D2-Pad2)")
     (add_net "Net-(D3-Pad2)")
+    (add_net "Net-(D4-Pad1)")
     (add_net "Net-(J3-Pad1)")
     (add_net "Net-(J4-Pad1)")
@@
   (module Project's_libs:SOIC127P1032X265-16N (layer B.Cu)
     (at 100.5 89.5 180)
-    (fp_text reference U1 (at -2.675 6.062) (layer B.SilkS)
-      (effects (font (size 1 1) (thickness 0.015)) (justify mirror))
+    (fp_text reference U1 (at -2.37 6.062) (layer B.SilkS)
+      (effects (font (size 1.016 1.016) (thickness 0.25)) (justify mirror))
     )
     (fp_text value DS3231 (at 6.85 -6.062) (layer B.Fab)
@@
       (at (xyz 0 0 0))
       (scale (xyz 1 1 1))
+      (rotate (xyz 0 0 0))
+    )
+  )
+  (module LEDs:LED_D5.0mm-4 (layer F.Cu)
+    (at 130.915001 32.485001)
+    (descr "LED, diameter 5.0mm, 2 pins, diameter 5.0mm, 3 pins, diameter 5.0mm, 4 pins, http://www.kingbright.com/attachments/file/psearch/000/00/00/L-154A4SUREQBFZGEW(Ver.9A).pdf")
+    (tags "LED diameter 5.0mm 2 pins diameter 5.0mm 3 pins diameter 5.0mm 4 pins")
+    (fp_text reference D4 (at 1.905 -3.96) (layer F.SilkS)
+      (effects (font (size 1 1) (thickness 0.15)))
+    )
+    (fp_text value Status_LEDs (at 1.905 3.96) (layer F.Fab)
+      (effects (font (size 1 1) (thickness 0.15)))
+    )
+    (fp_line (start 5.15 -3.25) (end -1.35 -3.25) (layer F.CrtYd) (width 0.05))
+    (fp_line (start 5.15 3.25) (end 5.15 -3.25) (layer F.CrtYd) (width 0.05))
+    (fp_line (start -1.35 3.25) (end 5.15 3.25) (layer F.CrtYd) (width 0.05))
+    (fp_line (start -1.35 -3.25) (end -1.35 3.25) (layer F.CrtYd) (width 0.05))
+    (fp_line (start -0.655 1.08) (end -0.655 1.545) (layer F.SilkS) (width 0.12))
+    (fp_line (start -0.655 -1.545) (end -0.655 -1.08) (layer F.SilkS) (width 0.12))
+    (fp_line (start -0.595 -1.469694) (end -0.595 1.469694) (layer F.Fab) (width 0.1))
+    (fp_circle (center 1.905 0) (end 4.405 0) (layer F.Fab) (width 0.1))
+    (fp_arc (start 1.905 0) (end -0.349684 1.08) (angle -128.8) (layer F.SilkS) (width 0.12))
+    (fp_arc (start 1.905 0) (end -0.349684 -1.08) (angle 128.8) (layer F.SilkS) (width 0.12))
+    (fp_arc (start 1.905 0) (end -0.655 1.54483) (angle -127.7) (layer F.SilkS) (width 0.12))
+    (fp_arc (start 1.905 0) (end -0.655 -1.54483) (angle 127.7) (layer F.SilkS) (width 0.12))
+    (fp_arc (start 1.905 0) (end -0.595 -1.469694) (angle 299.1) (layer F.Fab) (width 0.1))
+    (pad 4 thru_hole oval (at 3.81 0) (size 1.07 1.8) (drill 0.9) (layers *.Cu *.Mask))
+    (pad 3 thru_hole oval (at 2.54 0) (size 1.07 1.8) (drill 0.9) (layers *.Cu *.Mask))
+    (pad 2 thru_hole oval (at 1.27 0) (size 1.07 1.8) (drill 0.9) (layers *.Cu *.Mask))
+    (pad 1 thru_hole rect (at 0 0) (size 1.07 1.8) (drill 0.9) (layers *.Cu *.Mask)
+      (net 30 "Net-(D4-Pad1)"))
+    (model ${KISYS3DMOD}/LEDs.3dshapes/LED_D5.0mm-4.wrl
+      (at (xyz 0 0 0))
+      (scale (xyz 0.393701 0.393701 0.393701))
+      (rotate (xyz 0 0 0))
+    )
+  )
+  (module Resistors_SMD:R_1206 (layer F.Cu)
+    (at 139.265001 30.345001)
+    (descr "Resistor SMD 1206, reflow soldering, Vishay (see dcrcw.pdf)")
+    (tags "resistor 1206")
+    (attr smd)
+    (fp_text reference R11 (at 0 -1.85) (layer F.SilkS)
+      (effects (font (size 1 1) (thickness 0.15)))
+    )
+    (fp_text value 330Ω (at 0 1.95) (layer F.Fab)
+      (effects (font (size 1 1) (thickness 0.15)))
+    )
+    (fp_line (start 2.15 1.1) (end -2.15 1.1) (layer F.CrtYd) (width 0.05))
+    (fp_line (start 2.15 1.1) (end 2.15 -1.11) (layer F.CrtYd) (width 0.05))
+    (fp_line (start -2.15 -1.11) (end -2.15 1.1) (layer F.CrtYd) (width 0.05))
+    (fp_line (start -2.15 -1.11) (end 2.15 -1.11) (layer F.CrtYd) (width 0.05))
+    (fp_line (start -1 -1.07) (end 1 -1.07) (layer F.SilkS) (width 0.12))
+    (fp_line (start 1 1.07) (end -1 1.07) (layer F.SilkS) (width 0.12))
+    (fp_line (start -1.6 -0.8) (end 1.6 -0.8) (layer F.Fab) (width 0.1))
+    (fp_line (start 1.6 -0.8) (end 1.6 0.8) (layer F.Fab) (width 0.1))
+    (fp_line (start 1.6 0.8) (end -1.6 0.8) (layer F.Fab) (width 0.1))
+    (fp_line (start -1.6 0.8) (end -1.6 -0.8) (layer F.Fab) (width 0.1))
+    (fp_text user %R (at 0 0) (layer F.Fab)
+      (effects (font (size 0.7 0.7) (thickness 0.105)))
+    )
+    (pad 2 smd rect (at 1.45 0) (size 0.9 1.7) (layers F.Cu F.Paste F.Mask)
+      (net 1 GND))
+    (pad 1 smd rect (at -1.45 0) (size 0.9 1.7) (layers F.Cu F.Paste F.Mask)
+      (net 30 "Net-(D4-Pad1)"))
+    (model ${KISYS3DMOD}/Resistors_SMD.3dshapes/R_1206.wrl
+      (at (xyz 0 0 0))
+      (scale (xyz 1 1 1))

Commit message: Update
Parts:
- moved J4 147.0 mm to (96.8, 104.8), turned to 180 degrees
- moved J3 125.6 mm to (108.0, 104.8), turned to 180 degrees
- moved J1 105.0 mm to (119.1, 104.8), turned to 180 degrees
- moved U1 19.3 mm to (81.5, 86.4)
- moved BT1 19.1 mm to (81.5, 78.7), turned to 0 degrees
Changed lines of the file:
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@@
   )
   (module Morfeas_RPi_hat:CH252032LF (layer F.Cu)
-    (at 100.5 77.5 270)
+    (at 81.45 78.74)
     (descr CH25-2032LF-1)
     (tags "Undefined or Miscellaneous")
-    (fp_text reference BT1 (at -5 20) (layer F.SilkS)
+    (fp_text reference BT1 (at -5 20 -270) (layer F.SilkS)
       (effects (font (size 1.27 1.27) (thickness 0.254)))
     )
-    (fp_text value Battery_Cell (at 0 14.5 90) (layer F.SilkS) hide
+    (fp_text value Battery_Cell (at 0 14.5) (layer F.SilkS) hide
       (effects (font (size 1.27 1.27) (thickness 0.254)))
     )
@@
     (fp_arc (start 0 6) (end -11.4 6) (angle -180) (layer F.SilkS) (width 0.1))
     (fp_arc (start 0 6) (end 11.4 6) (angle -180) (layer F.SilkS) (width 0.1))
-    (pad 1 thru_hole circle (at 0 0 270) (size 1.65 1.65) (drill 1.1) (layers *.Cu *.Mask)
+    (pad 1 thru_hole circle (at 0 0) (size 1.65 1.65) (drill 1.1) (layers *.Cu *.Mask)
       (net 2 "Net-(BT1-Pad1)"))
-    (pad 2 thru_hole circle (at 0 20 270) (size 1.65 1.65) (drill 1.1) (layers *.Cu *.Mask)
+    (pad 2 thru_hole circle (at 0 20) (size 1.65 1.65) (drill 1.1) (layers *.Cu *.Mask)
       (net 1 GND))
     (model ${KIPRJMOD}/Project's_libs/STEP/CH25-2032LF_approx.step
@@
   )
   (module Morfeas_RPi_hat:SPTH_V1,5 (layer F.Cu)
-    (at 209.537001 51.445001)
+    (at 119.07 104.76 180)
     (fp_text reference J1 (at -3.5 -13) (layer F.SilkS)
       (effects (font (size 1 1) (thickness 0.15)))
@@
     (fp_line (start 5.5 -12) (end 5.5 1.5) (layer F.SilkS) (width 0.15))
     (fp_line (start -5.5 -12) (end 5.5 -12) (layer F.SilkS) (width 0.15))
-    (pad 3 thru_hole oval (at 3.5 0) (size 1.905 2.54) (drill 1.143 (offset 0 -0.381)) (layers *.Cu *.Mask)
-      (net 1 GND))
-    (pad 2 thru_hole oval (at 0 0) (size 1.905 2.54) (drill 1.143 (offset 0 -0.381)) (layers *.Cu *.Mask)
+    (pad 3 thru_hole oval (at 3.5 0 180) (size 1.905 2.54) (drill 1.143 (offset 0 -0.381)) (layers *.Cu *.Mask)
+      (net 1 GND))
+    (pad 2 thru_hole oval (at 0 0 180) (size 1.905 2.54) (drill 1.143 (offset 0 -0.381)) (layers *.Cu *.Mask)
       (net 15 +24V))
-    (pad 1 thru_hole oval (at -3.5 0) (size 1.905 2.54) (drill 1.143 (offset 0 -0.381)) (layers *.Cu *.Mask)
+    (pad 1 thru_hole oval (at -3.5 0 180) (size 1.905 2.54) (drill 1.143 (offset 0 -0.381)) (layers *.Cu *.Mask)
       (net 15 +24V))
-    (pad 3 thru_hole roundrect (at 3.5 -7) (size 1.905 2.54) (drill 1.143) (layers *.Cu *.Mask) (roundrect_rratio 0.5)
-      (net 1 GND))
-    (pad 2 thru_hole roundrect (at 0 -7) (size 1.905 2.54) (drill 1.143) (layers *.Cu *.Mask) (roundrect_rratio 0.5)
+    (pad 3 thru_hole roundrect (at 3.5 -7 180) (size 1.905 2.54) (drill 1.143) (layers *.Cu *.Mask) (roundrect_rratio 0.5)
+      (net 1 GND))
+    (pad 2 thru_hole roundrect (at 0 -7 180) (size 1.905 2.54) (drill 1.143) (layers *.Cu *.Mask) (roundrect_rratio 0.5)
       (net 15 +24V))
-    (pad 1 thru_hole roundrect (at -3.5 -7) (size 1.905 2.54) (drill 1.143) (layers *.Cu *.Mask) (roundrect_rratio 0.5)
+    (pad 1 thru_hole roundrect (at -3.5 -7 180) (size 1.905 2.54) (drill 1.143) (layers *.Cu *.Mask) (roundrect_rratio 0.5)
       (net 15 +24V))
     (model ${KIPRJMOD}/Project's_libs/STEP/pxc_1823641_05_SPT-THR-1-5-3-H-3-5-P20-R32_3D.step
@@
   )
   (module Morfeas_RPi_hat:SPTH_V1,5 (layer F.Cu)
-    (at 221.687001 51.445001)
+    (at 107.95 104.76 180)
     (fp_text reference J3 (at -3.5 -13) (layer F.SilkS)
       (effects (font (size 1 1) (thickness 0.15)))
@@
     (fp_line (start 5.5 -12) (end 5.5 1.5) (layer F.SilkS) (width 0.15))
     (fp_line (start -5.5 -12) (end 5.5 -12) (layer F.SilkS) (width 0.15))
-    (pad 3 thru_hole oval (at 3.5 0) (size 1.905 2.54) (drill 1.143 (offset 0 -0.381)) (layers *.Cu *.Mask)
-      (net 24 "Net-(J3-Pad1)"))
-    (pad 2 thru_hole oval (at 0 0) (size 1.905 2.54) (drill 1.143 (offset 0 -0.381)) (layers *.Cu *.Mask)
-      (net 24 "Net-(J3-Pad1)"))
-    (pad 1 thru_hole oval (at -3.5 0) (size 1.905 2.54) (drill 1.143 (offset 0 -0.381)) (layers *.Cu *.Mask)
-      (net 24 "Net-(J3-Pad1)"))
-    (pad 3 thru_hole roundrect (at 3.5 -7) (size 1.905 2.54) (drill 1.143) (layers *.Cu *.Mask) (roundrect_rratio 0.5)
-      (net 24 "Net-(J3-Pad1)"))
-    (pad 2 thru_hole roundrect (at 0 -7) (size 1.905 2.54) (drill 1.143) (layers *.Cu *.Mask) (roundrect_rratio 0.5)
-      (net 24 "Net-(J3-Pad1)"))
-    (pad 1 thru_hole roundrect (at -3.5 -7) (size 1.905 2.54) (drill 1.143) (layers *.Cu *.Mask) (roundrect_rratio 0.5)
+    (pad 3 thru_hole oval (at 3.5 0 180) (size 1.905 2.54) (drill 1.143 (offset 0 -0.381)) (layers *.Cu *.Mask)
+      (net 24 "Net-(J3-Pad1)"))
+    (pad 2 thru_hole oval (at 0 0 180) (size 1.905 2.54) (drill 1.143 (offset 0 -0.381)) (layers *.Cu *.Mask)
+      (net 24 "Net-(J3-Pad1)"))
+    (pad 1 thru_hole oval (at -3.5 0 180) (size 1.905 2.54) (drill 1.143 (offset 0 -0.381)) (layers *.Cu *.Mask)
+      (net 24 "Net-(J3-Pad1)"))
+    (pad 3 thru_hole roundrect (at 3.5 -7 180) (size 1.905 2.54) (drill 1.143) (layers *.Cu *.Mask) (roundrect_rratio 0.5)
+      (net 24 "Net-(J3-Pad1)"))
+    (pad 2 thru_hole roundrect (at 0 -7 180) (size 1.905 2.54) (drill 1.143) (layers *.Cu *.Mask) (roundrect_rratio 0.5)
+      (net 24 "Net-(J3-Pad1)"))
+    (pad 1 thru_hole roundrect (at -3.5 -7 180) (size 1.905 2.54) (drill 1.143) (layers *.Cu *.Mask) (roundrect_rratio 0.5)
       (net 24 "Net-(J3-Pad1)"))
     (model ${KIPRJMOD}/Project's_libs/STEP/pxc_1823641_05_SPT-THR-1-5-3-H-3-5-P20-R32_3D.step
@@
   )
   (module Morfeas_RPi_hat:SPTH_V1,5 (layer F.Cu)
-    (at 233.837001 51.445001)
+    (at 96.83 104.76 180)
     (fp_text reference J4 (at -3.5 -13) (layer F.SilkS)
       (effects (font (size 1 1) (thickness 0.15)))
@@
     (fp_line (start 5.5 -12) (end 5.5 1.5) (layer F.SilkS) (width 0.15))
     (fp_line (start -5.5 -12) (end 5.5 -12) (layer F.SilkS) (width 0.15))
-    (pad 3 thru_hole oval (at 3.5 0) (size 1.905 2.54) (drill 1.143 (offset 0 -0.381)) (layers *.Cu *.Mask)
-      (net 25 "Net-(J4-Pad1)"))
-    (pad 2 thru_hole oval (at 0 0) (size 1.905 2.54) (drill 1.143 (offset 0 -0.381)) (layers *.Cu *.Mask)
-      (net 25 "Net-(J4-Pad1)"))
-    (pad 1 thru_hole oval (at -3.5 0) (size 1.905 2.54) (drill 1.143 (offset 0 -0.381)) (layers *.Cu *.Mask)
-      (net 25 "Net-(J4-Pad1)"))
-    (pad 3 thru_hole roundrect (at 3.5 -7) (size 1.905 2.54) (drill 1.143) (layers *.Cu *.Mask) (roundrect_rratio 0.5)
-      (net 25 "Net-(J4-Pad1)"))
-    (pad 2 thru_hole roundrect (at 0 -7) (size 1.905 2.54) (drill 1.143) (layers *.Cu *.Mask) (roundrect_rratio 0.5)
-      (net 25 "Net-(J4-Pad1)"))
-    (pad 1 thru_hole roundrect (at -3.5 -7) (size 1.905 2.54) (drill 1.143) (layers *.Cu *.Mask) (roundrect_rratio 0.5)
+    (pad 3 thru_hole oval (at 3.5 0 180) (size 1.905 2.54) (drill 1.143 (offset 0 -0.381)) (layers *.Cu *.Mask)
+      (net 25 "Net-(J4-Pad1)"))
+    (pad 2 thru_hole oval (at 0 0 180) (size 1.905 2.54) (drill 1.143 (offset 0 -0.381)) (layers *.Cu *.Mask)
+      (net 25 "Net-(J4-Pad1)"))
+    (pad 1 thru_hole oval (at -3.5 0 180) (size 1.905 2.54) (drill 1.143 (offset 0 -0.381)) (layers *.Cu *.Mask)
+      (net 25 "Net-(J4-Pad1)"))
+    (pad 3 thru_hole roundrect (at 3.5 -7 180) (size 1.905 2.54) (drill 1.143) (layers *.Cu *.Mask) (roundrect_rratio 0.5)
+      (net 25 "Net-(J4-Pad1)"))
+    (pad 2 thru_hole roundrect (at 0 -7 180) (size 1.905 2.54) (drill 1.143) (layers *.Cu *.Mask) (roundrect_rratio 0.5)
+      (net 25 "Net-(J4-Pad1)"))
+    (pad 1 thru_hole roundrect (at -3.5 -7 180) (size 1.905 2.54) (drill 1.143) (layers *.Cu *.Mask) (roundrect_rratio 0.5)
       (net 25 "Net-(J4-Pad1)"))
     (model ${KIPRJMOD}/Project's_libs/STEP/pxc_1823641_05_SPT-THR-1-5-3-H-3-5-P20-R32_3D.step
@@
   )
   (module Project's_libs:SOIC127P1032X265-16N (layer B.Cu)
-    (at 100.5 89.5 180)
+    (at 81.45 86.36 180)
     (fp_text reference U1 (at -2.37 6.062) (layer B.SilkS)
       (effects (font (size 1.016 1.016) (thickness 0.25)) (justify mirror))
