File: src/Morfeas_RPi_Hat/Hardware/Morfeas_Rpi_Hat.kicad_pcb (KiCad board)
At the start: 2 copper layers, 65 x 56 mm, 49 parts, among them J1 Power IN, J2 RPi_header, J3 CAN0_Power+, J4 CAN1_Power+, J5 RS_232, Q1 SUM110P06, Q2 SUM110P06, U1 DS3231, U2 TSR2-2450, U3 TLV70433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

Commit message: Update
Parts:
- D4: footprint LEDs:LED_D5.0mm-4 -> LED_THT:LED_D5.0mm-4_RGB
- R11: footprint Resistors_SMD:R_1206 -> Resistor_SMD:R_1206_3216Metric
- moved J5 4.84 mm to (152.4, 34.8)
Changed lines of the file:
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@@
-(kicad_pcb (version 20171130) (host pcbnew "(5.1.5)-3")
+(kicad_pcb (version 20171130) (host pcbnew 5.1.5+dfsg1-2)
   (general
     (thickness 1.6)
@@
   )
   (module Connectors_Molex:Molex_KK-6410-03_03x2.54mm_Straight (layer F.Cu)
-    (at 157.099 35.941)
+    (at 152.4 34.798)
     (descr "Connector Headers with Friction Lock, 22-27-2031, http://www.molex.com/pdm_docs/sd/022272021_sd.pdf")
     (tags "connector molex kk_6410 22-27-2031")
@@
       (effects (font (size 1 1) (thickness 0.15)))
     )
-    (fp_text user %R (at 2.54 0) (layer F.Fab)
+    (fp_text user %R (at -3.937 1.397) (layer F.Fab)
       (effects (font (size 1 1) (thickness 0.15)))
     )
@@
     )
   )
-  (module LEDs:LED_D5.0mm-4 (layer F.Cu)
+  (module LED_THT:LED_D5.0mm-4_RGB (layer F.Cu)
     (at 130.915001 32.485001)
     (descr "LED, diameter 5.0mm, 2 pins, diameter 5.0mm, 3 pins, diameter 5.0mm, 4 pins, http://www.kingbright.com/attachments/file/psearch/000/00/00/L-154A4SUREQBFZGEW(Ver.9A).pdf")
-    (tags "LED diameter 5.0mm 2 pins diameter 5.0mm 3 pins diameter 5.0mm 4 pins")
+    (tags "LED diameter 5.0mm 2 pins diameter 5.0mm 3 pins diameter 5.0mm 4 pins RGB RGBLED")
     (fp_text reference D4 (at 1.905 -3.96) (layer F.SilkS)
       (effects (font (size 1 1) (thickness 0.15)))
@@
       (effects (font (size 1 1) (thickness 0.15)))
     )
+    (fp_arc (start 1.905 0) (end -0.595 -1.469694) (angle 299.1) (layer F.Fab) (width 0.1))
+    (fp_arc (start 1.905 0) (end -0.655 -1.54483) (angle 127.7) (layer F.SilkS) (width 0.12))
+    (fp_arc (start 1.905 0) (end -0.655 1.54483) (angle -127.7) (layer F.SilkS) (width 0.12))
+    (fp_arc (start 1.905 0) (end -0.349684 -1.08) (angle 128.8) (layer F.SilkS) (width 0.12))
+    (fp_arc (start 1.905 0) (end -0.349684 1.08) (angle -128.8) (layer F.SilkS) (width 0.12))
+    (fp_circle (center 1.905 0) (end 4.405 0) (layer F.Fab) (width 0.1))
+    (fp_line (start -0.595 -1.469694) (end -0.595 1.469694) (layer F.Fab) (width 0.1))
+    (fp_line (start -0.655 -1.545) (end -0.655 -1.08) (layer F.SilkS) (width 0.12))
+    (fp_line (start -0.655 1.08) (end -0.655 1.545) (layer F.SilkS) (width 0.12))
+    (fp_line (start -1.35 -3.25) (end -1.35 3.25) (layer F.CrtYd) (width 0.05))
+    (fp_line (start -1.35 3.25) (end 5.15 3.25) (layer F.CrtYd) (width 0.05))
+    (fp_line (start 5.15 3.25) (end 5.15 -3.25) (layer F.CrtYd) (width 0.05))
     (fp_line (start 5.15 -3.25) (end -1.35 -3.25) (layer F.CrtYd) (width 0.05))
-    (fp_line (start 5.15 3.25) (end 5.15 -3.25) (layer F.CrtYd) (width 0.05))
-    (fp_line (start -1.35 3.25) (end 5.15 3.25) (layer F.CrtYd) (width 0.05))
-    (fp_line (start -1.35 -3.25) (end -1.35 3.25) (layer F.CrtYd) (width 0.05))
-    (fp_line (start -0.655 1.08) (end -0.655 1.545) (layer F.SilkS) (width 0.12))
-    (fp_line (start -0.655 -1.545) (end -0.655 -1.08) (layer F.SilkS) (width 0.12))
-    (fp_line (start -0.595 -1.469694) (end -0.595 1.469694) (layer F.Fab) (width 0.1))
-    (fp_circle (center 1.905 0) (end 4.405 0) (layer F.Fab) (width 0.1))
-    (fp_arc (start 1.905 0) (end -0.349684 1.08) (angle -128.8) (layer F.SilkS) (width 0.12))
-    (fp_arc (start 1.905 0) (end -0.349684 -1.08) (angle 128.8) (layer F.SilkS) (width 0.12))
-    (fp_arc (start 1.905 0) (end -0.655 1.54483) (angle -127.7) (layer F.SilkS) (width 0.12))
-    (fp_arc (start 1.905 0) (end -0.655 -1.54483) (angle 127.7) (layer F.SilkS) (width 0.12))
-    (fp_arc (start 1.905 0) (end -0.595 -1.469694) (angle 299.1) (layer F.Fab) (width 0.1))
-    (pad 4 thru_hole oval (at 3.81 0) (size 1.07 1.8) (drill 0.9) (layers *.Cu *.Mask))
-    (pad 3 thru_hole oval (at 2.54 0) (size 1.07 1.8) (drill 0.9) (layers *.Cu *.Mask))
-    (pad 2 thru_hole oval (at 1.27 0) (size 1.07 1.8) (drill 0.9) (layers *.Cu *.Mask))
+    (fp_text user %R (at 1.905 -3.96) (layer F.Fab)
+      (effects (font (size 1 1) (thickness 0.15)))
+    )
     (pad 1 thru_hole rect (at 0 0) (size 1.07 1.8) (drill 0.9) (layers *.Cu *.Mask)
       (net 30 "Net-(D4-Pad1)"))
-    (model ${KISYS3DMOD}/LEDs.3dshapes/LED_D5.0mm-4.wrl
-      (at (xyz 0 0 0))
-      (scale (xyz 0.393701 0.393701 0.393701))
-      (rotate (xyz 0 0 0))
-    )
-  )
-  (module Resistors_SMD:R_1206 (layer F.Cu)
+    (pad 2 thru_hole oval (at 1.27 0) (size 1.07 1.8) (drill 0.9) (layers *.Cu *.Mask))
+    (pad 3 thru_hole oval (at 2.54 0) (size 1.07 1.8) (drill 0.9) (layers *.Cu *.Mask))
+    (pad 4 thru_hole oval (at 3.81 0) (size 1.07 1.8) (drill 0.9) (layers *.Cu *.Mask))
+    (model ${KISYS3DMOD}/LED_THT.3dshapes/LED_D5.0mm-4_RGB.wrl
+      (at (xyz 0 0 0))
+      (scale (xyz 1 1 1))
+      (rotate (xyz 0 0 0))
+    )
+  )
+  (module Resistor_SMD:R_1206_3216Metric (layer F.Cu)
     (at 139.265001 30.345001)
-    (descr "Resistor SMD 1206, reflow soldering, Vishay (see dcrcw.pdf)")
-    (tags "resistor 1206")
-    (attr smd)
-    (fp_text reference R11 (at 0 -1.85) (layer F.SilkS)
-      (effects (font (size 1 1) (thickness 0.15)))
-    )
-    (fp_text value 330Ω (at 0 1.95) (layer F.Fab)
-      (effects (font (size 1 1) (thickness 0.15)))
-    )
-    (fp_line (start 2.15 1.1) (end -2.15 1.1) (layer F.CrtYd) (width 0.05))
-    (fp_line (start 2.15 1.1) (end 2.15 -1.11) (layer F.CrtYd) (width 0.05))
-    (fp_line (start -2.15 -1.11) (end -2.15 1.1) (layer F.CrtYd) (width 0.05))
-    (fp_line (start -2.15 -1.11) (end 2.15 -1.11) (layer F.CrtYd) (width 0.05))
-    (fp_line (start -1 -1.07) (end 1 -1.07) (layer F.SilkS) (width 0.12))
-    (fp_line (start 1 1.07) (end -1 1.07) (layer F.SilkS) (width 0.12))
+    (descr "Resistor SMD 1206 (3216 Metric), square (rectangular) end terminal, IPC_7351 nominal, (Body size source: http://www.tortai-tech.com/upload/download/2011102023233369053.pdf), generated with kicad-footprint-generator")
+    (tags resistor)
+    (attr smd)
+    (fp_text reference R11 (at 0 -1.82) (layer F.SilkS)
+      (effects (font (size 1 1) (thickness 0.15)))
+    )
+    (fp_text value 330Ω (at 0 1.82) (layer F.Fab)
+      (effects (font (size 1 1) (thickness 0.15)))
+    )
+    (fp_line (start -1.6 0.8) (end -1.6 -0.8) (layer F.Fab) (width 0.1))
     (fp_line (start -1.6 -0.8) (end 1.6 -0.8) (layer F.Fab) (width 0.1))
     (fp_line (start 1.6 -0.8) (end 1.6 0.8) (layer F.Fab) (width 0.1))
     (fp_line (start 1.6 0.8) (end -1.6 0.8) (layer F.Fab) (width 0.1))
-    (fp_line (start -1.6 0.8) (end -1.6 -0.8) (layer F.Fab) (width 0.1))
-    (fp_text user %R (at 0 0) (layer F.Fab)
-      (effects (font (size 0.7 0.7) (thickness 0.105)))
-    )
-    (pad 2 smd rect (at 1.45 0) (size 0.9 1.7) (layers F.Cu F.Paste F.Mask)
-      (net 1 GND))
-    (pad 1 smd rect (at -1.45 0) (size 0.9 1.7) (layers F.Cu F.Paste F.Mask)
+    (fp_line (start -0.602064 -0.91) (end 0.602064 -0.91) (layer F.SilkS) (width 0.12))
+    (fp_line (start -0.602064 0.91) (end 0.602064 0.91) (layer F.SilkS) (width 0.12))
+    (fp_line (start -2.28 1.12) (end -2.28 -1.12) (layer F.CrtYd) (width 0.05))
+    (fp_line (start -2.28 -1.12) (end 2.28 -1.12) (layer F.CrtYd) (width 0.05))
+    (fp_line (start 2.28 -1.12) (end 2.28 1.12) (layer F.CrtYd) (width 0.05))
+    (fp_line (start 2.28 1.12) (end -2.28 1.12) (layer F.CrtYd) (width 0.05))
+    (fp_text user %R (at 0 0) (layer F.Fab)
+      (effects (font (size 0.8 0.8) (thickness 0.12)))
+    )
+    (pad 1 smd roundrect (at -1.4 0) (size 1.25 1.75) (layers F.Cu F.Paste F.Mask) (roundrect_rratio 0.2)
       (net 30 "Net-(D4-Pad1)"))
-    (model ${KISYS3DMOD}/Resistors_SMD.3dshapes/R_1206.wrl
-      (at (xyz 0 0 0))
-      (scale (xyz 1 1 1))
+    (pad 2 smd roundrect (at 1.4 0) (size 1.25 1.75) (layers F.Cu F.Paste F.Mask) (roundrect_rratio 0.2)
+      (net 1 GND))
+    (model ${KISYS3DMOD}/Resistor_SMD.3dshapes/R_1206_3216Metric.wrl
+      (at (xyz 0 0 0))
+      (scale (xyz 1 1 1))

Commit message: Update
Parts:
- J5: footprint Connectors_Molex:Molex_KK-6410-03_03x2.54mm_Straight -> Connector_PinHeader_2.54mm:PinHeader_1x03_P2.54mm_Horizontal
Changed lines of the file:
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@@
-    )
-  )
-  (module Connectors_Molex:Molex_KK-6410-03_03x2.54mm_Straight (layer F.Cu)
-    (at 152.4 34.798)
-    (descr "Connector Headers with Friction Lock, 22-27-2031, http://www.molex.com/pdm_docs/sd/022272021_sd.pdf")
-    (tags "connector molex kk_6410 22-27-2031")
-    (fp_text reference J5 (at 1 -4.5) (layer F.SilkS)
-      (effects (font (size 1 1) (thickness 0.15)))
-    )
-    (fp_text value RS_232 (at 2.54 4.5) (layer F.Fab)
-      (effects (font (size 1 1) (thickness 0.15)))
-    )
-    (fp_text user %R (at -3.937 1.397) (layer F.Fab)
-      (effects (font (size 1 1) (thickness 0.15)))
-    )
-    (fp_line (start 7 3.5) (end -1.9 3.5) (layer F.CrtYd) (width 0.05))
-    (fp_line (start 7 -3.55) (end 7 3.5) (layer F.CrtYd) (width 0.05))
-    (fp_line (start -1.9 -3.55) (end 7 -3.55) (layer F.CrtYd) (width 0.05))
-    (fp_line (start -1.9 3.5) (end -1.9 -3.55) (layer F.CrtYd) (width 0.05))
-    (fp_line (start 5.88 -2.4) (end 5.88 -3.02) (layer F.SilkS) (width 0.12))
-    (fp_line (start 4.28 -2.4) (end 5.88 -2.4) (layer F.SilkS) (width 0.12))
-    (fp_line (start 4.28 -3.02) (end 4.28 -2.4) (layer F.SilkS) (width 0.12))
-    (fp_line (start 3.34 -2.4) (end 3.34 -3.02) (layer F.SilkS) (width 0.12))
-    (fp_line (start 1.74 -2.4) (end 3.34 -2.4) (layer F.SilkS) (width 0.12))
-    (fp_line (start 1.74 -3.02) (end 1.74 -2.4) (layer F.SilkS) (width 0.12))
-    (fp_line (start 0.8 -2.4) (end 0.8 -3.02) (layer F.SilkS) (width 0.12))
-    (fp_line (start -0.8 -2.4) (end 0.8 -2.4) (layer F.SilkS) (width 0.12))
-    (fp_line (start -0.8 -3.02) (end -0.8 -2.4) (layer F.SilkS) (width 0.12))
-    (fp_line (start 4.83 2.98) (end 4.83 1.98) (layer F.SilkS) (width 0.12))
-    (fp_line (start 0.25 2.98) (end 0.25 1.98) (layer F.SilkS) (width 0.12))
-    (fp_line (start 4.83 1.55) (end 5.08 1.98) (layer F.SilkS) (width 0.12))
-    (fp_line (start 0.25 1.55) (end 4.83 1.55) (layer F.SilkS) (width 0.12))
-    (fp_line (start 0 1.98) (end 0.25 1.55) (layer F.SilkS) (width 0.12))
-    (fp_line (start 5.08 1.98) (end 5.08 2.98) (layer F.SilkS) (width 0.12))
-    (fp_line (start 0 1.98) (end 5.08 1.98) (layer F.SilkS) (width 0.12))
-    (fp_line (start 0 2.98) (end 0 1.98) (layer F.SilkS) (width 0.12))
-    (fp_line (start 6.45 -3.02) (end -1.37 -3.02) (layer F.SilkS) (width 0.12))
-    (fp_line (start 6.45 2.98) (end 6.45 -3.02) (layer F.SilkS) (width 0.12))
-    (fp_line (start -1.37 2.98) (end 6.45 2.98) (layer F.SilkS) (width 0.12))
-    (fp_line (start -1.37 -3.02) (end -1.37 2.98) (layer F.SilkS) (width 0.12))
-    (fp_line (start 6.55 -3.12) (end -1.47 -3.12) (layer F.Fab) (width 0.12))
-    (fp_line (start 6.55 3.08) (end 6.55 -3.12) (layer F.Fab) (width 0.12))
-    (fp_line (start -1.47 3.08) (end 6.55 3.08) (layer F.Fab) (width 0.12))
-    (fp_line (start -1.47 -3.12) (end -1.47 3.08) (layer F.Fab) (width 0.12))
-    (pad 3 thru_hole oval (at 5.08 0) (size 2 2.6) (drill 1.2) (layers *.Cu *.Mask)
-      (net 1 GND))
-    (pad 2 thru_hole oval (at 2.54 0) (size 2 2.6) (drill 1.2) (layers *.Cu *.Mask)
-      (net 28 "Net-(J5-Pad2)"))
-    (pad 1 thru_hole rect (at 0 0) (size 2 2.6) (drill 1.2) (layers *.Cu *.Mask)
-      (net 29 "Net-(J5-Pad1)"))
-    (model ${KISYS3DMOD}/Connectors_Molex.3dshapes/Molex_KK-6410-03_03x2.54mm_Straight.wrl
-      (at (xyz 0 0 0))
-      (scale (xyz 1 1 1))
-      (rotate (xyz 0 0 0))
     )
   )
@@
       (at (xyz 0 0 0))
       (scale (xyz 1 1 1))
+      (rotate (xyz 0 0 0))
+    )
+  )
+  (module Connector_PinHeader_2.54mm:PinHeader_1x03_P2.54mm_Horizontal (layer F.Cu)
+    (at 152.4 34.798)
+    (descr "Through hole angled pin header, 1x03, 2.54mm pitch, 6mm pin length, single row")
+    (tags "Through hole angled pin header THT 1x03 2.54mm single row")
+    (fp_text reference J5 (at 4.385 -2.27) (layer F.SilkS)
+      (effects (font (size 1 1) (thickness 0.15)))
+    )
+    (fp_text value RS_232 (at 4.385 7.35) (layer F.Fab)
+      (effects (font (size 1 1) (thickness 0.15)))
+    )
+    (fp_line (start 2.135 -1.27) (end 4.04 -1.27) (layer F.Fab) (width 0.1))
+    (fp_line (start 4.04 -1.27) (end 4.04 6.35) (layer F.Fab) (width 0.1))
+    (fp_line (start 4.04 6.35) (end 1.5 6.35) (layer F.Fab) (width 0.1))
+    (fp_line (start 1.5 6.35) (end 1.5 -0.635) (layer F.Fab) (width 0.1))
+    (fp_line (start 1.5 -0.635) (end 2.135 -1.27) (layer F.Fab) (width 0.1))
+    (fp_line (start -0.32 -0.32) (end 1.5 -0.32) (layer F.Fab) (width 0.1))
+    (fp_line (start -0.32 -0.32) (end -0.32 0.32) (layer F.Fab) (width 0.1))
+    (fp_line (start -0.32 0.32) (end 1.5 0.32) (layer F.Fab) (width 0.1))
+    (fp_line (start 4.04 -0.32) (end 10.04 -0.32) (layer F.Fab) (width 0.1))
+    (fp_line (start 10.04 -0.32) (end 10.04 0.32) (layer F.Fab) (width 0.1))
+    (fp_line (start 4.04 0.32) (end 10.04 0.32) (layer F.Fab) (width 0.1))
+    (fp_line (start -0.32 2.22) (end 1.5 2.22) (layer F.Fab) (width 0.1))
+    (fp_line (start -0.32 2.22) (end -0.32 2.86) (layer F.Fab) (width 0.1))
+    (fp_line (start -0.32 2.86) (end 1.5 2.86) (layer F.Fab) (width 0.1))
+    (fp_line (start 4.04 2.22) (end 10.04 2.22) (layer F.Fab) (width 0.1))
+    (fp_line (start 10.04 2.22) (end 10.04 2.86) (layer F.Fab) (width 0.1))
+    (fp_line (start 4.04 2.86) (end 10.04 2.86) (layer F.Fab) (width 0.1))
+    (fp_line (start -0.32 4.76) (end 1.5 4.76) (layer F.Fab) (width 0.1))
+    (fp_line (start -0.32 4.76) (end -0.32 5.4) (layer F.Fab) (width 0.1))
+    (fp_line (start -0.32 5.4) (end 1.5 5.4) (layer F.Fab) (width 0.1))
+    (fp_line (start 4.04 4.76) (end 10.04 4.76) (layer F.Fab) (width 0.1))
+    (fp_line (start 10.04 4.76) (end 10.04 5.4) (layer F.Fab) (width 0.1))
+    (fp_line (start 4.04 5.4) (end 10.04 5.4) (layer F.Fab) (width 0.1))
+    (fp_line (start 1.44 -1.33) (end 1.44 6.41) (layer F.SilkS) (width 0.12))
+    (fp_line (start 1.44 6.41) (end 4.1 6.41) (layer F.SilkS) (width 0.12))
+    (fp_line (start 4.1 6.41) (end 4.1 -1.33) (layer F.SilkS) (width 0.12))
+    (fp_line (start 4.1 -1.33) (end 1.44 -1.33) (layer F.SilkS) (width 0.12))
+    (fp_line (start 4.1 -0.38) (end 10.1 -0.38) (layer F.SilkS) (width 0.12))
+    (fp_line (start 10.1 -0.38) (end 10.1 0.38) (layer F.SilkS) (width 0.12))
+    (fp_line (start 10.1 0.38) (end 4.1 0.38) (layer F.SilkS) (width 0.12))
+    (fp_line (start 4.1 -0.32) (end 10.1 -0.32) (layer F.SilkS) (width 0.12))
+    (fp_line (start 4.1 -0.2) (end 10.1 -0.2) (layer F.SilkS) (width 0.12))
+    (fp_line (start 4.1 -0.08) (end 10.1 -0.08) (layer F.SilkS) (width 0.12))
+    (fp_line (start 4.1 0.04) (end 10.1 0.04) (layer F.SilkS) (width 0.12))
+    (fp_line (start 4.1 0.16) (end 10.1 0.16) (layer F.SilkS) (width 0.12))
+    (fp_line (start 4.1 0.28) (end 10.1 0.28) (layer F.SilkS) (width 0.12))
+    (fp_line (start 1.11 -0.38) (end 1.44 -0.38) (layer F.SilkS) (width 0.12))
+    (fp_line (start 1.11 0.38) (end 1.44 0.38) (layer F.SilkS) (width 0.12))
+    (fp_line (start 1.44 1.27) (end 4.1 1.27) (layer F.SilkS) (width 0.12))
+    (fp_line (start 4.1 2.16) (end 10.1 2.16) (layer F.SilkS) (width 0.12))
+    (fp_line (start 10.1 2.16) (end 10.1 2.92) (layer F.SilkS) (width 0.12))
+    (fp_line (start 10.1 2.92) (end 4.1 2.92) (layer F.SilkS) (width 0.12))
+    (fp_line (start 1.042929 2.16) (end 1.44 2.16) (layer F.SilkS) (width 0.12))
+    (fp_line (start 1.042929 2.92) (end 1.44 2.92) (layer F.SilkS) (width 0.12))
+    (fp_line (start 1.44 3.81) (end 4.1 3.81) (layer F.SilkS) (width 0.12))
+    (fp_line (start 4.1 4.7) (end 10.1 4.7) (layer F.SilkS) (width 0.12))
+    (fp_line (start 10.1 4.7) (end 10.1 5.46) (layer F.SilkS) (width 0.12))
+    (fp_line (start 10.1 5.46) (end 4.1 5.46) (layer F.SilkS) (width 0.12))
+    (fp_line (start 1.042929 4.7) (end 1.44 4.7) (layer F.SilkS) (width 0.12))
+    (fp_line (start 1.042929 5.46) (end 1.44 5.46) (layer F.SilkS) (width 0.12))
+    (fp_line (start -1.27 0) (end -1.27 -1.27) (layer F.SilkS) (width 0.12))
+    (fp_line (start -1.27 -1.27) (end 0 -1.27) (layer F.SilkS) (width 0.12))
+    (fp_line (start -1.8 -1.8) (end -1.8 6.85) (layer F.CrtYd) (width 0.05))
+    (fp_line (start -1.8 6.85) (end 10.55 6.85) (layer F.CrtYd) (width 0.05))
+    (fp_line (start 10.55 6.85) (end 10.55 -1.8) (layer F.CrtYd) (width 0.05))
+    (fp_line (start 10.55 -1.8) (end -1.8 -1.8) (layer F.CrtYd) (width 0.05))
+    (fp_text user %R (at 2.77 2.54 90) (layer F.Fab)
+      (effects (font (size 1 1) (thickness 0.15)))
+    )
+    (pad 1 thru_hole rect (at 0 0) (size 1.7 1.7) (drill 1) (layers *.Cu *.Mask)
+      (net 29 "Net-(J5-Pad1)"))
+    (pad 2 thru_hole oval (at 0 2.54) (size 1.7 1.7) (drill 1) (layers *.Cu *.Mask)
+      (net 28 "Net-(J5-Pad2)"))
+    (pad 3 thru_hole oval (at 0 5.08) (size 1.7 1.7) (drill 1) (layers *.Cu *.Mask)
+      (net 1 GND))
+    (model ${KISYS3DMOD}/Connector_PinHeader_2.54mm.3dshapes/PinHeader_1x03_P2.54mm_Horizontal.wrl
+      (at (xyz 0 0 0))
+      (scale (xyz 1 1 1))
