File: src/Morfeas_RPi_Hat/Hardware/Morfeas_Rpi_Hat.kicad_pcb (KiCad board)
At the start: 2 copper layers, 65 x 56 mm, 49 parts, among them J1 Power IN, J2 RPi_header, J3 CAN0_Power+, J4 CAN1_Power+, J5 RS_232, Q1 SUM110P06, Q2 SUM110P06, U1 DS3231, U2 TSR2-2450, U3 TLV70433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

Commit message: Update
Connections:
- U6 pad 8: (no net) -> +3V3
- U6 pad 9: (no net) -> GND
- U7 pad 8: (no net) -> +3V3
- U7 pad 9: (no net) -> +3V3
Changed lines of the file:
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@@
     (pad 7 smd rect (at 2.1717 0.499999) (size 1.4224 0.2794) (layers F.Cu F.Paste F.Mask)
       (net 18 SDA))
-    (pad 8 smd rect (at 2.1717 0) (size 1.4224 0.2794) (layers F.Cu F.Paste F.Mask))
-    (pad 9 smd rect (at 2.1717 -0.499999) (size 1.4224 0.2794) (layers F.Cu F.Paste F.Mask))
+    (pad 8 smd rect (at 2.1717 0) (size 1.4224 0.2794) (layers F.Cu F.Paste F.Mask)
+      (net 10 +3V3))
+    (pad 9 smd rect (at 2.1717 -0.499999) (size 1.4224 0.2794) (layers F.Cu F.Paste F.Mask)
+      (net 1 GND))
     (pad 10 smd rect (at 2.1717 -1.000001) (size 1.4224 0.2794) (layers F.Cu F.Paste F.Mask)
       (net 10 +3V3))
@@
     (pad 10 smd rect (at 2.1717 -1.000001) (size 1.4224 0.2794) (layers F.Cu F.Paste F.Mask)
       (net 10 +3V3))
-    (pad 9 smd rect (at 2.1717 -0.499999) (size 1.4224 0.2794) (layers F.Cu F.Paste F.Mask))
-    (pad 8 smd rect (at 2.1717 0) (size 1.4224 0.2794) (layers F.Cu F.Paste F.Mask))
+    (pad 9 smd rect (at 2.1717 -0.499999) (size 1.4224 0.2794) (layers F.Cu F.Paste F.Mask)
+      (net 10 +3V3))
+    (pad 8 smd rect (at 2.1717 0) (size 1.4224 0.2794) (layers F.Cu F.Paste F.Mask)
+      (net 10 +3V3))
     (pad 7 smd rect (at 2.1717 0.499999) (size 1.4224 0.2794) (layers F.Cu F.Paste F.Mask)
       (net 18 SDA))

Commit message: Update Morfeas_RPi_hat
Parts:
- added C15: 100nf, Capacitors_SMD:C_0805, B.Cu at (88.1, 83.6)
- added R12: 1kΩ, Resistors_SMD:R_1206, B.Cu at (83.4, 78.2)
- added R13: 1kΩ, Resistors_SMD:R_1206, B.Cu at (94.9, 100.6)
- C1, C12, C13, C14, C2, C3, C9, R10, R11, R4, R6, R7, R8, R9, U6, U7: moved to B.Cu
- J5: footprint Connector_PinHeader_2.54mm:PinHeader_1x03_P2.54mm_Horizontal -> Pin_Headers:Pin_Header_Straight_1x03_Pitch2.54mm
- LED1: renamed from D4; footprint LED_THT:LED_D5.0mm-4_RGB -> Pin_Headers:Pin_Header_Straight_1x04_Pitch2.54mm
- moved C8 166.1 mm to (70.1, 73.2), turned to 90 degrees
- moved C10 153.4 mm to (77.5, 100.8)
- moved C7 152.4 mm to (87.6, 107.5), turned to 270 degrees
- moved C5 133.0 mm to (81.0, 100.8)
- moved U3 131.8 mm to (90.5, 72.4), turned to 270 degrees
- moved C9 125.6 mm to (84.3, 106.1), turned to 90 degrees
- moved R10 124.4 mm to (98.2, 72.9), turned to 180 degrees
- moved U5 123.7 mm to (73.7, 73.2), turned to 180 degrees
- moved U4 120.8 mm to (81.3, 106.0), turned to 270 degrees
- moved U7 119.2 mm to (99.7, 96.8), turned to 180 degrees
- moved C2 117.0 mm to (112.5, 78.4), turned to 270 degrees
- moved C4 116.7 mm to (84.5, 100.8)
- moved R7 114.8 mm to (125.0, 85.2), turned to 90 degrees
- moved C6 105.6 mm to (86.9, 72.8), turned to 270 degrees
- moved J5 104.1 mm to (84.5, 113.7), turned to 270 degrees
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Connections:
- J2 pad 29: (no net) -> R
- J2 pad 31: (no net) -> G
- J2 pad 33: (no net) -> B
- LED1 pad 2: (no net) -> R
- LED1 pad 3: (no net) -> G
- LED1 pad 4: (no net) -> B
Routing:
- net +3V3: track 0.00 -> 132.3 mm, vias 0 -> 7
- net SCL: track 0.00 -> 89.7 mm, vias 0 -> 1
- net SDA: track 0.00 -> 82.8 mm, vias 0 -> 1
- net GND: track 0.00 -> 75.2 mm, vias 0 -> 3
- net RXD: track 0.00 -> 55.5 mm
- net TXD: track 0.00 -> 54.8 mm
- net +5V: track 0.00 -> 52.6 mm, vias 0 -> 2
- net +24V: track 0.00 -> 48.0 mm, vias 0 -> 16
- net R: track 0.00 -> 29.0 mm
- net G: track 0.00 -> 23.5 mm
- net B: track 0.00 -> 19.2 mm
- net Net-(D2-Pad2): track 0.00 -> 19.0 mm
- net Net-(BT1-Pad1): track 0.00 -> 15.2 mm, vias 0 -> 1
- net Net-(D3-Pad2): track 0.00 -> 14.4 mm, vias 0 -> 1
- net Net-(Q1-Pad2): track 0.00 -> 13.7 mm, vias 0 -> 1
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- added copper zone on B.Cu, net +24V
- added copper zone on F.Cu, net +24V
- added copper zone on B.Cu, net GND
- added copper zone on F.Cu, net GND
- added copper zone on F.Cu, net Net-(J3-Pad1)
- added copper zone on F.Cu, net Net-(J4-Pad1)
- added copper zone on F.Cu, net Net-(Q1-Pad2)
- added copper zone on F.Cu, net Net-(Q2-Pad2)
Other:
- net class Default: clearance 0.2286 -> 0.127
- net class Power_24 removed
- net class Power_5 removed
- rule pad_to_mask_clearance: 0.051 -> 0.0762
- rule solder_mask_min_width: 0.25 -> 0.127
- rule trace_clearance: 0.2286 -> 0.127
- rule trace_min: 0.2 -> 0.127
- rule via_min_size: 0.4 -> 0.254
- board text added: "- + +"
- board text added: "C"
- board text added: "CAN0 +"
- board text added: "CAN1 +"
- board text added: "G RX TX"
- board text added: "Morfeas RPi Hat V1.0"
- board text added: "R G B"

Commit message: Update Morfeas_RPi_hat
Routing:
- net +5V: track 52.6 -> 61.7 mm, vias 2 -> 3
- net +3V3: track 132.3 -> 137.8 mm
- net Net-(C12-Pad2): track 7.01 -> 7.51 mm
Changed lines of the file:
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@@
     (thickness 1.6)
     (drawings 21)
-    (tracks 351)
+    (tracks 362)
     (zones 0)
     (modules 52)
@@
   )
   (layers
-    (0 F.Cu signal)
+    (0 F.Cu signal hide)
     (31 B.Cu signal)
     (32 B.Adhes user hide)
     (33 F.Adhes user hide)
-    (34 B.Paste user)
-    (35 F.Paste user)
-    (36 B.SilkS user)
-    (37 F.SilkS user)
+    (34 B.Paste user hide)
+    (35 F.Paste user hide)
+    (36 B.SilkS user hide)
+    (37 F.SilkS user hide)
     (38 B.Mask user)
-    (39 F.Mask user)
+    (39 F.Mask user hide)
     (40 Dwgs.User user)
     (41 Cmts.User user)
@@
   )
   (setup
-    (last_trace_width 1.27)
+    (last_trace_width 0.254)
     (user_trace_width 0.4064)
     (user_trace_width 0.635)
@@
   (segment (start 83.917 107.031) (end 85.09 107.031) (width 0.635) (layer B.Cu) (net 1) (status 10))
   (segment (start 85.078 106.922) (end 85.949 106.075) (width 0.635) (layer B.Cu) (net 1))
-  (via (at 103.124 70.104) (size 1.27) (drill 0.6) (layers F.Cu B.Cu) (net 1))
+  (via (at 102.616 70.612) (size 1.27) (drill 0.6) (layers F.Cu B.Cu) (net 1))
   (segment (start 99.076 63.23) (end 97.79 64.516) (width 0.4064) (layer B.Cu) (net 1) (status 10))
   (segment (start 99.23 63.23) (end 99.076 63.23) (width 0.4064) (layer B.Cu) (net 1) (status 30))
@@
   (segment (start 76.37 63.23) (end 78.91 63.23) (width 1.27) (layer B.Cu) (net 5) (status 30))
   (segment (start 107.696 71.12) (end 107.696 71.882) (width 0.635) (layer F.Cu) (net 5) (status 30))
-  (via (at 92.964 68.834) (size 1.27) (drill 0.6) (layers F.Cu B.Cu) (net 5))
-  (segment (start 92.964 68.834) (end 92.202 68.072) (width 1.27) (layer B.Cu) (net 5))
-  (segment (start 92.202 68.072) (end 90.424 68.072) (width 1.27) (layer B.Cu) (net 5))
-  (segment (start 92.964 68.834) (end 105.41 68.834) (width 0.635) (layer F.Cu) (net 5))
+  (via (at 95.25 68.834) (size 1.27) (drill 0.6) (layers F.Cu B.Cu) (net 5))
+  (segment (start 92.964 68.834) (end 105.41 68.834) (width 1.27) (layer F.Cu) (net 5))
   (segment (start 105.41 68.834) (end 107.696 71.12) (width 0.635) (layer F.Cu) (net 5) (status 20))
-  (segment (start 92.964 68.834) (end 91.186 68.834) (width 1.27) (layer B.Cu) (net 5))
   (segment (start 107.696 71.882) (end 105.156 71.882) (width 1.27) (layer B.Cu) (net 5) (status 30))
+  (segment (start 91.186 68.834) (end 92.964 68.834) (width 1.27) (layer B.Cu) (net 5))
+  (segment (start 94.742 68.072) (end 90.424 68.072) (width 1.27) (layer B.Cu) (net 5))
+  (segment (start 92.964 68.834) (end 93.218 68.834) (width 1.27) (layer B.Cu) (net 5))
+  (segment (start 95.504 68.834) (end 94.742 68.072) (width 1.27) (layer B.Cu) (net 5))
+  (segment (start 93.218 68.834) (end 95.504 68.834) (width 1.27) (layer B.Cu) (net 5))
+  (via (at 93.218 68.834) (size 1.27) (drill 0.6) (layers F.Cu B.Cu) (net 5))
+  (segment (start 91.186 68.834) (end 95.25 68.834) (width 1.27) (layer F.Cu) (net 5))
   (segment (start 83.185 102.235) (end 83.185 103.57) (width 0.635) (layer F.Cu) (net 6) (status 20))
   (segment (start 83.566 100.838) (end 83.566 101.854) (width 0.635) (layer F.Cu) (net 6) (status 10))
@@
   (via (at 86.868 69.85) (size 1.27) (drill 0.6) (layers F.Cu B.Cu) (net 10))
   (segment (start 86.868 71.374) (end 86.868 69.85) (width 0.635) (layer F.Cu) (net 10) (status 10))
-  (segment (start 97.5233 95.794999) (end 97.5233 96.795) (width 0.4064) (layer B.Cu) (net 10) (status 30))
-  (segment (start 97.5233 96.295001) (end 99.030999 96.295001) (width 0.4064) (layer B.Cu) (net 10) (status 10))
-  (via (at 99.030999 96.295001) (size 1.27) (drill 0.6) (layers F.Cu B.Cu) (net 10))
   (segment (start 99.030999 96.295001) (end 103.094999 96.295001) (width 0.635) (layer F.Cu) (net 10))
   (segment (start 103.094999 96.295001) (end 104.648 94.742) (width 0.635) (layer F.Cu) (net 10))
@@
   (via (at 89.662 101.6) (size 1.27) (drill 0.6) (layers F.Cu B.Cu) (net 10))
   (segment (start 90.678 100.584) (end 89.662 101.6) (width 0.635) (layer B.Cu) (net 10))
+  (via (at 99.030999 96.295001) (size 1.27) (drill 0.6) (layers F.Cu B.Cu) (net 10))
+  (segment (start 97.5233 96.295001) (end 99.030999 96.295001) (width 0.254) (layer B.Cu) (net 10))
+  (segment (start 98.530997 95.794999) (end 99.030999 96.295001) (width 0.254) (layer B.Cu) (net 10))
+  (segment (start 97.5233 95.794999) (end 98.530997 95.794999) (width 0.254) (layer B.Cu) (net 10))
+  (segment (start 98.531 96.795) (end 99.030999 96.295001) (width 0.254) (layer B.Cu) (net 10))
+  (segment (start 97.5233 96.795) (end 98.531 96.795) (width 0.254) (layer B.Cu) (net 10))
+  (segment (start 96.795 96.795) (end 96.295001 96.295001) (width 0.254) (layer B.Cu) (net 10))
+  (segment (start 97.5233 96.795) (end 96.795 96.795) (width 0.254) (layer B.Cu) (net 10))
+  (segment (start 96.229001 95.794999) (end 96.012 96.012) (width 0.254) (layer B.Cu) (net 10))
+  (segment (start 97.5233 95.794999) (end 96.229001 95.794999) (width 0.254) (layer B.Cu) (net 10))
   (segment (start 84.455 103.57) (end 84.455 105.029) (width 0.254) (layer F.Cu) (net 11) (status 10))
   (segment (start 84.455 105.029) (end 84.074 105.41) (width 0.254) (layer F.Cu) (net 11))
@@
   (segment (start 128.524 99.054) (end 128.524 98.298) (width 1.27) (layer F.Cu) (net 13) (status 10))
   (segment (start 128.524 98.298) (end 128.524 97.282) (width 1.27) (layer F.Cu) (net 13) (status 20))
-  (segment (start 104.629001 97.294999) (end 104.648 97.276) (width 0.4064) (layer B.Cu) (net 14) (status 30))
-  (segment (start 101.8667 97.294999) (end 104.629001 97.294999) (width 0.4064) (layer B.Cu) (net 14) (status 30))
   (segment (start 107.43 97.276) (end 107.442 97.288) (width 0.4064) (layer B.Cu) (net 14) (status 30))
   (segment (start 104.648 97.276) (end 107.43 97.276) (width 0.4064) (layer B.Cu) (net 14) (status 30))
   (segment (start 107.442 97.288) (end 107.442 98.709) (width 0.635) (layer B.Cu) (net 14) (status 30))
+  (segment (start 105.143001 97.294999) (end 105.156 97.282) (width 0.254) (layer B.Cu) (net 14))
+  (segment (start 101.8667 97.294999) (end 105.143001 97.294999) (width 0.254) (layer B.Cu) (net 14))
   (segment (start 95.504 72.898) (end 94.234 72.898) (width 0.635) (layer F.Cu) (net 15) (status 20))
   (segment (start 97.155 74.549) (end 95.504 72.898) (width 0.635) (layer F.Cu) (net 15))

Commit message: Update Morfeas_RPi_hat
Parts:
- added Open_Source_hardware1: Open Source Hardware, Symbols:OSHW-Logo2_7.3x6mm_SilkScreen, F.Cu at (129.3, 106.9)
- D1: footprint Diode_THT:D_DO-34_SOD68_P7.62mm_Horizontal -> Diodes_ThroughHole:D_DO-41_SOD81_P10.16mm_Horizontal
- moved R13 6.80 mm to (88.1, 100.2), turned to 90 degrees
- moved D1 1.02 mm to (110.0, 89.7)
- moved R6 0.77 mm to (107.4, 95.1)
- moved C12 0.51 mm to (107.4, 99.2)
- renumbered LED1 to D4
Routing:
- net Net-(R7-Pad1): track 10.6 -> 18.4 mm
- net GND: track 75.2 -> 81.8 mm
- net +3V3: track 137.8 -> 134.5 mm
- net Net-(C1-Pad1): track 6.10 -> 5.08 mm

Commit message: Update Morfeas_RPi_hat
Routing:
- net Net-(C12-Pad2): track 7.51 -> 12.1 mm

Commit message: Update
Parts:
- C15: footprint Capacitors_SMD:C_0805 -> Capacitor_SMD:C_0805_2012Metric
- D1: footprint Diodes_ThroughHole:D_DO-41_SOD81_P10.16mm_Horizontal -> Diode_THT:D_DO-41_SOD81_P10.16mm_Horizontal
- D4: footprint Pin_Headers:Pin_Header_Straight_1x04_Pitch2.54mm -> Connector_PinHeader_2.54mm:PinHeader_1x04_P2.54mm_Vertical
- J5: footprint Pin_Headers:Pin_Header_Straight_1x03_Pitch2.54mm -> Connector_PinHeader_2.54mm:PinHeader_1x03_P2.54mm_Vertical
- R12, R13: footprint Resistors_SMD:R_1206 -> Resistor_SMD:R_1206_3216Metric
- moved BT1 53.7 mm to (134.2, 95.9)
- moved C1 53.7 mm to (166.1, 88.3)
- moved C10 53.7 mm to (131.1, 103.4)
- moved C12 53.7 mm to (161.0, 101.8)
- moved C13 53.7 mm to (169.4, 96.1)
- moved C2 53.7 mm to (166.1, 80.9)
- moved C5 53.7 mm to (134.6, 103.4)
- moved D3 53.7 mm to (147.8, 75.4)
- moved J1 53.7 mm to (161.8, 107.3)
- moved J3 53.7 mm to (173.2, 107.3)
- moved J5 53.7 mm to (138.0, 116.2)
- moved R6 53.7 mm to (161.0, 97.7)
- moved R7 53.7 mm to (178.6, 87.8)
- moved U1 53.7 mm to (134.2, 88.3)
- moved U2 53.7 mm to (163.8, 74.4)
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
Commit message: Update Morfeas_RPi_Hat
Parts:
- added D5: NRVTSA4100ET3G, Morfeas_RPi_hat:DO-214AC(SMA), B.Cu at (178.8, 111.0)
- added D6: NRVTSA4100ET3G, Morfeas_RPi_hat:DO-214AC(SMA), B.Cu at (144.8, 111.0)
- moved Open_Source_hardware1 0.36 mm to (182.6, 109.2)
Routing:
- net +24V: track 48.0 -> 19.6 mm
- net Net-(D6-Pad1): track 7.51 -> 14.5 mm
- net Net-(D5-Pad1): track 6.14 -> 13.1 mm
- net GND: track 81.8 -> 81.3 mm
Other:
- rule trace_min: 0.127 -> 0.254
- rule via_min_size: 0.254 -> 1.016
- board text added: "CAN0 P+"
- board text added: "CAN1 P+"
- board text removed: "CAN0 +"
- board text removed: "CAN1 +"
