File: src/Morfeas_RPi_Hat/Hardware/Morfeas_Rpi_Hat.kicad_pcb (KiCad board)
At the start: 2 copper layers, 65 x 56 mm, 58 parts, among them J1 Con, J2 RPi_header, J5 RS_232, Q1 SUM110P06, Q2 SUM110P06, U1 DS3231, U2 TSR2-2450, U3 TLV70433, U4 SP3232, U5 24AA08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

Commit message: Update Morfeas_RPi_Hat files
Parts:
- removed G***: LOGO, Morfeas_RPi_Hat:Morfeas_logo
- added Morfeas_project_Logo1: Morfeas Project's Logo, Morfeas_RPi_Hat:Morfeas_logo, F.Cu at (164.8, 87.9)
- H1, H2, H3, H4: footprint MountingHole:MountingHole_3mm -> MountingHole:MountingHole_3.5mm
- Open_Source_hardware1: footprint Symbol:OSHW-Logo2_9.8x8mm_SilkScreen -> Symbol:OSHW-Logo2_7.3x6mm_SilkScreen
- U2: footprint Morfeas_RPi_hat:TSR2-2450 -> Morfeas_RPi_Hat:TSR2-2450
- U3: footprint Morfeas_RPi_hat:TLV70433DBVT -> Morfeas_RPi_Hat:TLV70433DBVT
Routing:
- net GND: track 86.3 -> 93.6 mm, vias 8 -> 9
- net +5V: track 63.2 -> 58.9 mm
- net +3V3: track 142.7 -> 143.9 mm

Commit message: Update Morfeas_RPi_Hat files
Parts:
- added Kicad_Logo: KiCad-Logo2_5mm_SilkScreen, Symbol:KiCad-Logo2_5mm_SilkScreen, B.Cu at (126.2, 103.6)
- BT1: footprint Morfeas_RPi_hat:CH252032LF -> Morfeas_RPi_Hat:CH252032LF

Commit message: Update Morfeas_RPi_Hat files
Parts:
- removed Kicad_Logo: KiCad-Logo2_5mm_SilkScreen, Symbol:KiCad-Logo2_5mm_SilkScreen
Routing:
- net GND: track 93.6 -> 87.1 mm, vias 9 -> 10

Commit message: Update Morfeas_RPi_Hat files
Routing:
- net +24V: track 47.4 -> 51.7 mm
- net +3V3: track 143.9 -> 142.5 mm
Changed lines of the file:
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@@
     (thickness 1.6)
     (drawings 27)
-    (tracks 439)
+    (tracks 440)
     (zones 0)
     (modules 58)
@@
     (39 F.Mask user)
     (40 Dwgs.User user)
-    (41 Cmts.User user)
+    (41 Cmts.User user hide)
     (42 Eco1.User user hide)
     (43 Eco2.User user hide)
@@
   )
   (setup
-    (last_trace_width 0.254)
+    (last_trace_width 1.27)
     (user_trace_width 0.4064)
     (user_trace_width 0.635)
@@
       (viasonmask true)
       (mode 1)
-      (useauxorigin true)
+      (useauxorigin false)
       (hpglpennumber 1)
       (hpglpenspeed 20)
@@
   (segment (start 124.714 72.39) (end 123.698 73.406) (width 0.635) (layer B.Cu) (net 10))
   (segment (start 140.462 72.39) (end 124.714 72.39) (width 0.635) (layer B.Cu) (net 10))
-  (via (at 141.732 82.296) (size 1.27) (drill 0.6) (layers F.Cu B.Cu) (net 10))
-  (segment (start 141.732 82.296) (end 141.732 85.106) (width 0.635) (layer B.Cu) (net 10) (status 20))
   (segment (start 170.815 97.155) (end 170.688 97.028) (width 0.254) (layer B.Cu) (net 10))
   (via (at 170.815 97.155) (size 1.27) (drill 0.6) (layers F.Cu B.Cu) (net 10))
   (segment (start 138.43 80.772) (end 141.732 80.772) (width 0.635) (layer B.Cu) (net 10) (status 10))
   (segment (start 141.732 75.184) (end 141.732 80.772) (width 0.635) (layer B.Cu) (net 10))
-  (segment (start 141.732 80.772) (end 141.732 82.296) (width 0.635) (layer B.Cu) (net 10))
   (via (at 143.256 104.14) (size 1.27) (drill 0.6) (layers F.Cu B.Cu) (net 10))
   (segment (start 150.389 99.335) (end 149.889001 98.835001) (width 0.254) (layer B.Cu) (net 10))
@@
   (via (at 148.844 97.028) (size 1.27) (drill 0.6) (layers F.Cu B.Cu) (net 10))
   (segment (start 141.732 104.14) (end 143.256 104.14) (width 0.635) (layer B.Cu) (net 10) (status 10))
-  (segment (start 143.002 82.296) (end 141.732 82.296) (width 0.635) (layer F.Cu) (net 10))
   (segment (start 158.242 97.282) (end 156.688999 98.835001) (width 0.635) (layer F.Cu) (net 10))
-  (segment (start 144.526 94.742) (end 144.526 83.82) (width 0.635) (layer F.Cu) (net 10))
-  (segment (start 144.526 83.82) (end 143.002 82.296) (width 0.635) (layer F.Cu) (net 10))
   (segment (start 143.256 104.14) (end 144.526 102.87) (width 0.635) (layer F.Cu) (net 10))
   (segment (start 144.809001 98.835001) (end 144.526 98.552) (width 0.635) (layer F.Cu) (net 10))
   (segment (start 144.526 102.87) (end 144.526 98.552) (width 0.635) (layer F.Cu) (net 10))
-  (segment (start 144.526 98.552) (end 144.526 94.742) (width 0.635) (layer F.Cu) (net 10))
   (segment (start 159.264 96.26) (end 158.242 97.282) (width 0.635) (layer B.Cu) (net 10))
   (segment (start 166.618 96.26) (end 159.264 96.26) (width 0.635) (layer B.Cu) (net 10))
@@
   (segment (start 142.494 72.39) (end 140.462 72.39) (width 0.4064) (layer F.Cu) (net 10))
   (segment (start 143.133998 73.029998) (end 142.494 72.39) (width 0.4064) (layer F.Cu) (net 10))
+  (segment (start 141.732 83.82) (end 141.732 85.106) (width 0.635) (layer B.Cu) (net 10))
+  (via (at 141.732 83.82) (size 1.27) (drill 0.6) (layers F.Cu B.Cu) (net 10))
+  (segment (start 141.732 80.772) (end 141.732 83.82) (width 0.635) (layer B.Cu) (net 10))
+  (segment (start 143.256 83.82) (end 141.732 83.82) (width 0.635) (layer F.Cu) (net 10))
+  (segment (start 144.526 98.552) (end 144.526 85.09) (width 0.635) (layer F.Cu) (net 10))
+  (segment (start 144.526 85.09) (end 143.256 83.82) (width 0.635) (layer F.Cu) (net 10))
   (segment (start 138.049 106.11) (end 138.049 107.569) (width 0.254) (layer F.Cu) (net 11) (status 10))
   (segment (start 138.049 107.569) (end 137.668 107.95) (width 0.254) (layer F.Cu) (net 11))
@@
   (segment (start 149.352 75.438) (end 150.114 76.2) (width 1.27) (layer F.Cu) (net 15))
   (segment (start 150.114 76.2) (end 150.622 76.708) (width 1.27) (layer F.Cu) (net 15))
+  (segment (start 172.212 75.438) (end 172.212 77.216) (width 1.27) (layer F.Cu) (net 15))
+  (segment (start 172.212 76.708) (end 170.434 78.486) (width 1.27) (layer F.Cu) (net 15))
   (segment (start 151.1173 99.834999) (end 149.847001 99.834999) (width 0.254) (layer B.Cu) (net 16) (status 10))
   (segment (start 149.847001 99.834999) (end 149.352 100.33) (width 0.254) (layer B.Cu) (net 16))
@@
     (polygon
       (pts
-        (xy 161.544 85.842287) (xy 158.496 82.926144) (xy 158.496 77.216) (xy 161.544 77.216)
+        (xy 161.544 86.106) (xy 158.242 82.804) (xy 158.242 77.216) (xy 161.544 77.216)
       )
     )

Commit message: Update Morfeas_RPi_Hat files
Parts:
- moved R12 1.02 mm to (137.0, 79.8)
Routing:
- net GND: track 87.1 -> 93.8 mm, vias 10 -> 14
- net /CAN1_P+: track 35.1 -> 38.7 mm
- net +5V: track 58.9 -> 61.4 mm
- net SDA: track 82.6 -> 85.0 mm
- net +3V3: track 142.5 -> 143.3 mm
Other:
- rule pad_to_mask_clearance: 0.0762 -> 0.127

Commit message: Update Morfeas_RPi_Hat files
Routing:
- net SCL: track 89.7 -> 108.3 mm
- net +24V: track 51.7 -> 66.9 mm
- net /CAN0_P+: track 27.8 -> 33.0 mm
- net +3V3: track 143.3 -> 144.1 mm

Commit message: Update Morfeas_RPi_Hat files
Routing:
- net +24V: track 66.9 -> 69.9 mm
- net GND: track 93.8 -> 92.6 mm

Commit message: Update Morfeas_RPi_Hat files
Routing:
- net +3V3: track 144.1 -> 148.5 mm
Changed lines of the file:
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@@
     (thickness 1.6)
     (drawings 27)
-    (tracks 475)
+    (tracks 482)
     (zones 0)
     (modules 58)
@@
   (segment (start 143.256 104.14) (end 144.526 102.87) (width 0.635) (layer F.Cu) (net 10))
   (segment (start 144.809001 98.835001) (end 144.526 98.552) (width 0.635) (layer F.Cu) (net 10))
-  (segment (start 144.526 102.87) (end 144.526 98.552) (width 0.635) (layer F.Cu) (net 10))
   (segment (start 159.264 96.26) (end 158.242 97.282) (width 0.635) (layer B.Cu) (net 10))
   (segment (start 166.618 96.26) (end 159.264 96.26) (width 0.635) (layer B.Cu) (net 10))
@@
   (segment (start 148.844 97.028) (end 147.066 98.806) (width 0.635) (layer F.Cu) (net 10))
   (segment (start 147.544999 98.835001) (end 147.066 98.806) (width 0.635) (layer F.Cu) (net 10))
-  (segment (start 147.066 98.806) (end 144.809001 98.835001) (width 0.635) (layer F.Cu) (net 10))
   (segment (start 156.688999 98.835001) (end 150.622 98.806) (width 0.635) (layer F.Cu) (net 10))
   (segment (start 148.844 97.028) (end 150.622 98.806) (width 0.635) (layer F.Cu) (net 10))
@@
   (via (at 141.732 83.82) (size 1.27) (drill 0.6) (layers F.Cu B.Cu) (net 10))
   (segment (start 143.256 83.82) (end 141.732 83.82) (width 0.635) (layer F.Cu) (net 10))
-  (segment (start 144.526 98.552) (end 144.526 85.09) (width 0.635) (layer F.Cu) (net 10))
   (segment (start 144.526 85.09) (end 143.256 83.82) (width 0.635) (layer F.Cu) (net 10))
   (segment (start 139.381 110.998) (end 139.319 111.06) (width 0.635) (layer F.Cu) (net 10))
@@
   (segment (start 181.61 97.028) (end 180.34 97.028) (width 0.635) (layer F.Cu) (net 10))
   (segment (start 180.34 97.028) (end 178.308 99.06) (width 0.635) (layer F.Cu) (net 10))
+  (segment (start 146.313667 98.815667) (end 145.551667 98.815667) (width 0.635) (layer F.Cu) (net 10))
+  (segment (start 145.551667 98.815667) (end 144.526 97.79) (width 0.635) (layer F.Cu) (net 10))
+  (segment (start 146.313667 98.815667) (end 144.809001 98.835001) (width 0.635) (layer F.Cu) (net 10))
+  (segment (start 147.066 98.806) (end 146.313667 98.815667) (width 0.635) (layer F.Cu) (net 10))
+  (segment (start 144.526 97.79) (end 144.526 85.09) (width 0.635) (layer F.Cu) (net 10))
+  (segment (start 144.526 98.552) (end 144.526 97.79) (width 0.635) (layer F.Cu) (net 10))
+  (segment (start 145.532333 98.815667) (end 144.526 99.822) (width 0.635) (layer F.Cu) (net 10))
+  (segment (start 146.313667 98.815667) (end 145.532333 98.815667) (width 0.635) (layer F.Cu) (net 10))
+  (segment (start 144.526 102.87) (end 144.526 99.822) (width 0.635) (layer F.Cu) (net 10))
+  (segment (start 144.526 99.822) (end 144.526 98.552) (width 0.635) (layer F.Cu) (net 10))
   (via (at 135.89 108.458) (size 1.27) (drill 0.6) (layers F.Cu B.Cu) (net 11))
   (segment (start 136.398 107.696) (end 135.89 108.204) (width 0.635) (layer B.Cu) (net 11))
