File: src/Morfeas_RPi_Hat/Hardware/_autosave-Morfeas_Rpi_Hat.kicad_pcb (KiCad board)
At the start: 2 copper layers, 65 x 56 mm, 53 parts, among them J1 Con, J2 RPi_header, J5 RS_232, Q1 SUM110P06, Q2 SUM110P06, U1 DS3231, U2 TSR2-2450, U3 TLV70433, U4 SP3232, U5 24AA08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

Commit message: Update Morfeas_RPi_Hat
Parts:
- moved D5 6.25 mm to (172.6, 111.5)
Routing:
- net Net-(D5-Pad1): track 13.1 -> 22.3 mm
- net Net-(D6-Pad1): track 23.2 -> 31.4 mm
- removed copper zone on F.Cu, net Net-(D5-Pad1)
Changed lines of the file:
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@@
     (thickness 1.6)
     (drawings 21)
-    (tracks 377)
+    (tracks 382)
     (zones 0)
     (modules 53)
@@
   )
   (module "Morfeas_RPi_hat:DO-214AC(SMA)" (layer B.Cu)
-    (at 178.816 110.998)
+    (at 172.58792 111.506)
     (descr "DO-214AC (SMA)  PACKAGE.")
     (tags "DO-214AC SMA")
@@
   (segment (start 183.896 76.708) (end 183.896 72.644) (width 0.4064) (layer B.Cu) (net 31) (status 10))
   (segment (start 183.896 72.644) (end 181.864 70.612) (width 0.4064) (layer B.Cu) (net 31))
-  (segment (start 176.728 107.3) (end 176.728 114.3) (width 2.54) (layer B.Cu) (net 32))
+  (segment (start 174.244 103.632) (end 174.244 102.235) (width 1.27) (layer F.Cu) (net 32))
+  (segment (start 174.244 103.632) (end 172.212 103.632) (width 2.54) (layer F.Cu) (net 32))
+  (segment (start 170.624 105.22) (end 170.624 107.514) (width 2.54) (layer F.Cu) (net 32))
+  (segment (start 172.212 103.632) (end 170.624 105.22) (width 2.54) (layer F.Cu) (net 32))
+  (segment (start 170.624 115.714) (end 170.624 107.514) (width 2.54) (layer B.Cu) (net 32))
   (segment (start 149.606 107.532) (end 149.606 115.57) (width 2.54) (layer B.Cu) (net 33))
   (segment (start 149.624 107.514) (end 149.606 107.532) (width 2.54) (layer B.Cu) (net 33))
@@
   (segment (start 149.624 105.138) (end 151.892 102.87) (width 2.54) (layer F.Cu) (net 33))
   (segment (start 151.892 102.87) (end 153.924 102.87) (width 2.54) (layer F.Cu) (net 33))
+  (segment (start 149.624 107.514) (end 149.624 115.714) (width 2.54) (layer F.Cu) (net 33))
   (zone (net 1) (net_name GND) (layer B.Cu) (hatch edge 0.508)
     (connect_pads yes (clearance 0.762))
@@
       )
     )
-  )
-  (zone (net 32) (net_name "Net-(D5-Pad1)") (layer F.Cu) (hatch edge 0.508)
-    (priority 1)
-    (connect_pads yes (clearance 0.762))
-    (min_thickness 0.254)
-    (fill yes (arc_segments 32) (thermal_gap 0.508) (thermal_bridge_width 0.508))
-    (polygon
-      (pts
-        (xy 178.054 116.078) (xy 168.402 116.078) (xy 168.402 105.156) (xy 171.958 101.6) (xy 178.054 101.6)
-      )
-    )
